Commit message: Wheels and base_link elements connected and moving.

File: urdf/common_properties.xacro (robot description, xacro)
@@ -32,4 +32,5 @@
   <xacro:property name="base_axis_length" value="${motor_length + wheel_width}"/>
   <xacro:property name="base_axis_mass" value="1.0"/>
+  <xacro:property name="gear_ratio" value="2"/>
   <xacro:macro name="cylinder_inertia" params="m r h">
     <inertia ixx="${m*(3*r*r+h*h)/12}" ixy="0" ixz="0"

File: urdf/gazebo.urdf.xacro (robot description, xacro)
@@ -7,6 +7,6 @@
     <gazebo reference="${name}">
       <material>Gazebo/Black</material>
-      <mu1>0.8</mu1>
-      <mu2>0.8</mu2>
+      <mu1>1.0</mu1>
+      <mu2>1.0</mu2>
       <kp>1000000.0</kp>
       <kd>100.0</kd>
@@ -14,6 +14,21 @@
       <maxVel>1.0</maxVel>
       <fdir1>1 0 0</fdir1>
-      <slip1>0.05</slip1>
-      <slip2>0.05</slip2>
+      <surface>
+        <friction>
+          <ode>
+            <mu>1.0</mu>
+            <mu2>1.0</mu2>
+            <fdir1>1 0 0</fdir1>
+          </ode>
+        </friction>
+        <contact>
+          <ode>
+            <kp>1e6</kp>
+            <kd>100.0</kd>
+            <max_vel>1.0</max_vel>
+            <min_depth>0.001</min_depth>
+          </ode>
+        </contact>
+      </surface>
     </gazebo>
   </xacro:macro>

File: urdf/shelfbot.urdf.xacro (robot description, xacro)
@@ -91,23 +91,31 @@
     <dynamics damping="0.1" friction="0.1"/>
   </joint>
-  <joint name="joint_wheel_front_left" type="fixed">
+  <joint name="joint_wheel_front_left" type="continuous">
     <parent link="base_axis_front_left"/>
     <child link="wheel_front_left"/>
     <origin xyz="0 0 -${motor_length/2}" rpy="0 0 0"/>
+    <axis xyz="0 0 1"/>
+    <mimic joint="joint_base_axis_front_left" multiplier="${gear_ratio}" offset="0"/>
   </joint>
-  <joint name="joint_wheel_front_right" type="fixed">
+  <joint name="joint_wheel_front_right" type="continuous">
     <parent link="base_axis_front_right"/>
     <child link="wheel_front_right"/>
     <origin xyz="0 0 ${motor_length/2}" rpy="0 0 0"/>
+    <axis xyz="0 0 1"/>
+    <mimic joint="joint_base_axis_front_right" multiplier="${gear_ratio}" offset="0"/>
   </joint>
-  <joint name="joint_wheel_back_left" type="fixed">
+  <joint name="joint_wheel_back_left" type="continuous">
     <parent link="base_axis_back_left"/>
     <child link="wheel_back_left"/>
     <origin xyz="0 0 -${motor_length/2}" rpy="0 0 0"/>
+    <axis xyz="0 0 1"/>
+    <mimic joint="joint_base_axis_back_left" multiplier="${gear_ratio}" offset="0"/>
   </joint>
-  <joint name="joint_wheel_back_right" type="fixed">
+  <joint name="joint_wheel_back_right" type="continuous">
     <parent link="base_axis_back_right"/>
     <child link="wheel_back_right"/>
     <origin xyz="0 0 ${motor_length/2}" rpy="0 0 0"/>
+    <axis xyz="0 0 1"/>
+    <mimic joint="joint_base_axis_back_right" multiplier="${gear_ratio}" offset="0"/>
   </joint>
   <xacro:camera name="camera" width="${camera_width}" length="${camera_length}" height="${camera_height}" radius="${camera_lens_radius}"/>

Commit message: Publishing odom and tf2 messages.

File: urdf/common_properties.xacro (robot description, xacro)
@@ -16,5 +16,5 @@
   <xacro:property name="base_length" value="0.7"/>
   <xacro:property name="base_height" value="0.2"/>
-  <xacro:property name="base_mass" value="20.0"/>
+  <xacro:property name="base_mass" value="50.0"/>
   <xacro:property name="motor_radius" value="0.05"/>
   <xacro:property name="motor_length" value="0.2"/>
@@ -22,5 +22,5 @@
   <xacro:property name="wheel_radius" value="0.2"/>
   <xacro:property name="wheel_width" value="0.05"/>
-  <xacro:property name="wheel_mass" value="3.0"/>
+  <xacro:property name="wheel_mass" value="5.0"/>
   <xacro:property name="camera_width" value="0.2"/>
   <xacro:property name="camera_length" value="0.2"/>

File: urdf/gazebo.urdf.xacro (robot description, xacro)
@@ -7,6 +7,6 @@
     <gazebo reference="${name}">
       <material>Gazebo/Black</material>
-      <mu1>1.0</mu1>
-      <mu2>1.0</mu2>
+      <mu1>0.8</mu1>
+      <mu2>0.8</mu2>
       <kp>1000000.0</kp>
       <kd>100.0</kd>
@@ -17,6 +17,6 @@
         <friction>
           <ode>
-            <mu>1.0</mu>
-            <mu2>1.0</mu2>
+            <mu>0.8</mu>
+            <mu2>0.8</mu2>
             <fdir1>1 0 0</fdir1>
           </ode>
@@ -110,4 +110,5 @@
   <gazebo>
     <plugin name="gazebo_ros2_control" filename="libgazebo_ros2_control.so">
+      <robotNamespace>/</robotNamespace>
       <parameters>$(find shelfbot)/config/four_wheel_drive_controller.yaml</parameters>
     </plugin>

File: urdf/shelfbot.urdf.xacro (robot description, xacro)
@@ -94,5 +94,5 @@
     <parent link="base_axis_front_left"/>
     <child link="wheel_front_left"/>
-    <origin xyz="${base_axis_length - wheel_width} 0 0" rpy="0 0 0"/>
+    <origin xyz="${base_axis_length/2} 0 0" rpy="0 0 0"/>
     <axis xyz="1 0 0"/>
     <mimic joint="joint_base_axis_front_left" multiplier="${gear_ratio}" offset="0"/>
@@ -101,5 +101,5 @@
     <parent link="base_axis_front_right"/>
     <child link="wheel_front_right"/>
-    <origin xyz="${base_axis_length - wheel_width} 0 0" rpy="0 0 0"/>
+    <origin xyz="${base_axis_length/2} 0 0" rpy="0 0 0"/>
     <axis xyz="1 0 0"/>
     <mimic joint="joint_base_axis_front_right" multiplier="${gear_ratio}" offset="0"/>
@@ -108,5 +108,5 @@
     <parent link="base_axis_back_left"/>
     <child link="wheel_back_left"/>
-    <origin xyz="${base_axis_length - wheel_width} 0 0" rpy="0 0 0"/>
+    <origin xyz="${base_axis_length/2} 0 0" rpy="0 0 0"/>
     <axis xyz="1 0 0"/>
     <mimic joint="joint_base_axis_back_left" multiplier="${gear_ratio}" offset="0"/>
@@ -115,5 +115,5 @@
     <parent link="base_axis_back_right"/>
     <child link="wheel_back_right"/>
-    <origin xyz="${base_axis_length - wheel_width} 0 0" rpy="0 0 0"/>
+    <origin xyz="${base_axis_length/2} 0 0" rpy="0 0 0"/>
     <axis xyz="1 0 0"/>
     <mimic joint="joint_base_axis_back_right" multiplier="${gear_ratio}" offset="0"/>

Commit message: Adding indicator_box to troubleshoot physics.

File: urdf/common_properties.xacro (robot description, xacro)
@@ -12,4 +12,7 @@
   <material name="metallic_gray">
     <color rgba="0.66 0.66 0.66 1.0"/>
+  </material>
+  <material name="red">
+    <color rgba="1.0 0.0 0.0 1.0"/>
   </material>
   <xacro:property name="base_width" value="0.5"/>

File: urdf/gazebo.urdf.xacro (robot description, xacro)
@@ -4,19 +4,22 @@
     <material>Gazebo/Gold</material>
   </gazebo>
+  <gazebo reference="indicator_box">
+    <material>Gazebo/Red</material>
+  </gazebo>
   <xacro:macro name="wheel_gazebo" params="name">
     <gazebo reference="${name}">
       <material>Gazebo/Black</material>
-      <mu1>0.8</mu1>
-      <mu2>0.8</mu2>
+      <mu1>1.8</mu1>
+      <mu2>1.8</mu2>
       <kp>1000000.0</kp>
       <kd>100.0</kd>
       <minDepth>0.001</minDepth>
-      <maxVel>1.0</maxVel>
+      <maxVel>1000.0</maxVel>
       <fdir1>1 0 0</fdir1>
       <surface>
         <friction>
           <ode>
-            <mu>0.8</mu>
-            <mu2>0.8</mu2>
+            <mu>1.8</mu>
+            <mu2>1.8</mu2>
             <fdir1>1 0 0</fdir1>
           </ode>
@@ -26,5 +29,5 @@
             <kp>1e6</kp>
             <kd>100.0</kd>
-            <max_vel>1.0</max_vel>
+            <max_vel>100.0</max_vel>
             <min_depth>0.001</min_depth>
           </ode>
@@ -104,8 +107,4 @@
     </transmission>
   </xacro:macro>
-  <xacro:wheel_transmission name="joint_wheel_front_left"/>
-  <xacro:wheel_transmission name="joint_wheel_front_right"/>
-  <xacro:wheel_transmission name="joint_wheel_back_left"/>
-  <xacro:wheel_transmission name="joint_wheel_back_right"/>
   <gazebo>
     <plugin name="gazebo_ros2_control" filename="libgazebo_ros2_control.so">

File: urdf/shelfbot.urdf.xacro (robot description, xacro)
@@ -7,4 +7,5 @@
   <xacro:include filename="$(find shelfbot)/urdf/base_axis.xacro"/>
   <xacro:include filename="$(find shelfbot)/urdf/gazebo.urdf.xacro"/>
+  <xacro:include filename="$(find shelfbot)/urdf/box.xacro"/>
   <link name="base_footprint"/>
   <link name="base_link">
@@ -43,4 +44,5 @@
   <xacro:wheel name="wheel_back_left" radius="${wheel_radius}" width="${wheel_width}"/>
   <xacro:wheel name="wheel_back_right" radius="${wheel_radius}" width="${wheel_width}"/>
+  <xacro:box name="indicator_box" parent_link="wheel_front_right"/>
   <joint name="joint_motor_front_left" type="fixed">
     <parent link="base_link"/>
@@ -91,31 +93,23 @@
     <dynamics damping="0.1" friction="0.1"/>
   </joint>
-  <joint name="joint_wheel_front_left" type="continuous">
+  <joint name="joint_wheel_front_left" type="fixed">
     <parent link="base_axis_front_left"/>
     <child link="wheel_front_left"/>
     <origin xyz="${base_axis_length/2} 0 0" rpy="0 0 0"/>
-    <axis xyz="1 0 0"/>
-    <mimic joint="joint_base_axis_front_left" multiplier="${gear_ratio}" offset="0"/>
   </joint>
-  <joint name="joint_wheel_front_right" type="continuous">
+  <joint name="joint_wheel_front_right" type="fixed">
     <parent link="base_axis_front_right"/>
     <child link="wheel_front_right"/>
     <origin xyz="${base_axis_length/2} 0 0" rpy="0 0 0"/>
-    <axis xyz="1 0 0"/>
-    <mimic joint="joint_base_axis_front_right" multiplier="${gear_ratio}" offset="0"/>
   </joint>
-  <joint name="joint_wheel_back_left" type="continuous">
+  <joint name="joint_wheel_back_left" type="fixed">
     <parent link="base_axis_back_left"/>
     <child link="wheel_back_left"/>
     <origin xyz="${base_axis_length/2} 0 0" rpy="0 0 0"/>
-    <axis xyz="1 0 0"/>
-    <mimic joint="joint_base_axis_back_left" multiplier="${gear_ratio}" offset="0"/>
   </joint>
-  <joint name="joint_wheel_back_right" type="continuous">
+  <joint name="joint_wheel_back_right" type="fixed">
     <parent link="base_axis_back_right"/>
     <child link="wheel_back_right"/>
     <origin xyz="${base_axis_length/2} 0 0" rpy="0 0 0"/>
-    <axis xyz="1 0 0"/>
-    <mimic joint="joint_base_axis_back_right" multiplier="${gear_ratio}" offset="0"/>
   </joint>
   <xacro:camera name="camera" width="${camera_width}" length="${camera_length}" height="${camera_height}" radius="${camera_lens_radius}"/>

Commit message: Organizing common_properties and the yaml.

File: urdf/common_properties.xacro (robot description, xacro)
@@ -1,4 +1,6 @@
 <?xml version="1.0"?>
 <robot xmlns:xacro="http://www.ros.org/wiki/xacro">
+  <xacro:property name="config_file" value="$(find shelfbot)/config/four_wheel_drive_controller.yaml" />
+  <xacro:property name="config" value="${xacro.load_yaml(config_file)}" />
   <material name="golden_brown">
     <color rgba="0.87 0.72 0.53 1.0"/>
@@ -16,24 +18,24 @@
     <color rgba="1.0 0.0 0.0 1.0"/>
   </material>
-  <xacro:property name="base_width" value="0.5"/>
-  <xacro:property name="base_length" value="0.7"/>
-  <xacro:property name="base_height" value="0.2"/>
-  <xacro:property name="base_mass" value="50.0"/>
-  <xacro:property name="motor_radius" value="0.05"/>
-  <xacro:property name="motor_length" value="0.2"/>
-  <xacro:property name="motor_mass" value="2.0"/>
-  <xacro:property name="wheel_radius" value="0.2"/>
-  <xacro:property name="wheel_width" value="0.05"/>
-  <xacro:property name="wheel_mass" value="5.0"/>
-  <xacro:property name="camera_width" value="0.2"/>
-  <xacro:property name="camera_length" value="0.2"/>
-  <xacro:property name="camera_height" value="0.1"/>
-  <xacro:property name="camera_lens_radius" value="0.05"/>
-  <xacro:property name="camera_mount_height" value="0.5"/>
-  <xacro:property name="camera_mass" value="0.5"/>
-  <xacro:property name="base_axis_radius" value="0.02"/>
-  <xacro:property name="base_axis_length" value="${motor_length + wheel_width}"/>
-  <xacro:property name="base_axis_mass" value="1.0"/>
-  <xacro:property name="gear_ratio" value="2"/>
+  <xacro:property name="base_width" value="${config['four_wheel_drive_controller']['ros__parameters']['base_width']}"/>
+  <xacro:property name="base_length" value="${config['four_wheel_drive_controller']['ros__parameters']['base_length']}"/>
+  <xacro:property name="base_height" value="${config['four_wheel_drive_controller']['ros__parameters']['base_height']}"/>
+  <xacro:property name="base_mass" value="${config['four_wheel_drive_controller']['ros__parameters']['base_mass']}"/>
+  <xacro:property name="motor_radius" value="${config['four_wheel_drive_controller']['ros__parameters']['motor_radius']}"/>
+  <xacro:property name="motor_length" value="${config['four_wheel_drive_controller']['ros__parameters']['motor_length']}"/>
+  <xacro:property name="motor_mass" value="${config['four_wheel_drive_controller']['ros__parameters']['motor_mass']}"/>
+  <xacro:property name="wheel_radius" value="${config['four_wheel_drive_controller']['ros__parameters']['wheel_radius']}"/>
+  <xacro:property name="wheel_width" value="${config['four_wheel_drive_controller']['ros__parameters']['wheel_width']}"/>
+  <xacro:property name="wheel_mass" value="${config['four_wheel_drive_controller']['ros__parameters']['wheel_mass']}"/>
+  <xacro:property name="camera_width" value="${config['four_wheel_drive_controller']['ros__parameters']['camera_width']}"/>
+  <xacro:property name="camera_length" value="${config['four_wheel_drive_controller']['ros__parameters']['camera_length']}"/>
+  <xacro:property name="camera_height" value="${config['four_wheel_drive_controller']['ros__parameters']['camera_height']}"/>
+  <xacro:property name="camera_lens_radius" value="${config['four_wheel_drive_controller']['ros__parameters']['camera_lens_radius']}"/>
+  <xacro:property name="camera_mount_height" value="${config['four_wheel_drive_controller']['ros__parameters']['camera_mount_height']}"/>
+  <xacro:property name="camera_mass" value="${config['four_wheel_drive_controller']['ros__parameters']['camera_mass']}"/>
+  <xacro:property name="base_axis_radius" value="${config['four_wheel_drive_controller']['ros__parameters']['base_axis_radius']}"/>
+  <xacro:property name="base_axis_length" value="${config['four_wheel_drive_controller']['ros__parameters']['base_axis_length']}"/>
+  <xacro:property name="base_axis_mass" value="${config['four_wheel_drive_controller']['ros__parameters']['base_axis_mass']}"/>
+  <xacro:property name="gear_ratio" value="${config['four_wheel_drive_controller']['ros__parameters']['gear_ratio']}"/>
   <xacro:macro name="cylinder_inertia" params="m r h">
     <inertia ixx="${m*(3*r*r+h*h)/12}" ixy="0" ixz="0"
