Commit message: Matching XACRO, URDF files to match the real robot.

File: urdf/base_axis.xacro (robot description, xacro)
@@ -1,5 +1,5 @@
 <?xml version="1.0"?>
 <robot xmlns:xacro="http://www.ros.org/wiki/xacro">
-  <xacro:macro name="motor" params="name length radius mass ixx ixy ixz iyy iyz izz">
+  <xacro:macro name="base_axis" params="name length radius">
     <link name="${name}">
       <visual>
@@ -7,5 +7,5 @@
           <cylinder length="${length}" radius="${radius}"/>
         </geometry>
-        <material name="metallic_gray"/>
+        <material name="dark_red"/>
       </visual>
       <collision>
@@ -14,9 +14,4 @@
         </geometry>
       </collision>
-      <inertial>
-        <mass value="${mass}"/>
-        <origin xyz="0 0 0" rpy="0 0 0"/>
-        <inertia ixx="${ixx}" ixy="${ixy}" ixz="${ixz}" iyy="${iyy}" iyz="${iyz}" izz="${izz}"/>
-      </inertial>
     </link>
   </xacro:macro>

File: urdf/camera.xacro (robot description, xacro)
@@ -9,5 +9,6 @@
           <cylinder length="0.05" radius="${radius}"/>
         </geometry>
-        <material name="gray"/>
+        <!-- Fixed: Changed material from "gray" to "metallic_gray" -->
+        <material name="metallic_gray"/>
       </visual>
       <collision>

File: urdf/common_properties.xacro (robot description, xacro)
@@ -2,9 +2,15 @@
 <robot xmlns:xacro="http://www.ros.org/wiki/xacro">
   <!-- Material Definitions -->
-  <material name="gray">
-    <color rgba="0.5 0.5 0.5 1.0"/>
+  <material name="golden_brown">
+    <color rgba="0.87 0.72 0.53 1.0"/>
   </material>
-  <material name="black">
-    <color rgba="0 0 0 1.0"/>
+  <material name="metallic_dark_lead">
+    <color rgba="0.33 0.33 0.33 1.0"/>
+  </material>
+  <material name="dark_red">
+    <color rgba="0.55 0.0 0.0 1.0"/>
+  </material>
+  <material name="metallic_gray">
+    <color rgba="0.66 0.66 0.66 1.0"/>
   </material>
   <!-- Common dimensions for motors and wheels -->
@@ -14,5 +20,5 @@
   <xacro:property name="motor_radius" value="0.05"/>
   <xacro:property name="motor_length" value="0.2"/>
-  <xacro:property name="wheel_radius" value="0.1"/>
+  <xacro:property name="wheel_radius" value="0.2"/>
   <xacro:property name="wheel_width" value="0.05"/>
   <xacro:property name="camera_width" value="0.2"/>
@@ -21,3 +27,5 @@
   <xacro:property name="camera_lens_radius" value="0.05"/>
   <xacro:property name="camera_mount_height" value="0.5"/>
+  <xacro:property name="base_axis_radius" value="0.02"/>
+  <xacro:property name="base_axis_length" value="${motor_length + wheel_width}"/>
 </robot>

File: urdf/fixed_joint.xacro (robot description, xacro)
@@ -1,9 +1,9 @@
 <?xml version="1.0"?>
 <robot xmlns:xacro="http://www.ros.org/wiki/xacro">
-  <xacro:macro name="fixed_joint" params="name parent child origin_xyz">
+  <xacro:macro name="fixed_joint" params="name parent child origin_xyz origin_rpy='0 0 0'">
     <joint name="${name}" type="fixed">
       <parent link="${parent}"/>
       <child link="${child}"/>
-      <origin xyz="${origin_xyz}" rpy="0 0 0"/>
+      <origin xyz="${origin_xyz}" rpy="${origin_rpy}"/>
     </joint>
   </xacro:macro>

File: urdf/shelfbot.urdf.xacro (robot description, xacro)
@@ -8,4 +8,7 @@
   <xacro:include filename="$(find shelfbot)/urdf/fixed_joint.xacro"/>
   <xacro:include filename="$(find shelfbot)/urdf/revolute_joint.xacro"/>
+  <xacro:include filename="$(find shelfbot)/urdf/base_axis.xacro"/>
+  <!-- Base Footprint Link -->
+  <link name="base_footprint"/>
   <!-- Base Link -->
   <link name="base_link">
@@ -14,21 +17,18 @@
         <box size="${base_width} ${base_length} ${base_height}"/>
       </geometry>
-      <material name="gray"/>
+      <material name="golden_brown"/>
     </visual>
   </link>
-  <!-- Base Footprint Link -->
-  <link name="base_footprint">
-    <visual>
-      <geometry>
-        <box size="${base_width} ${base_length} 0.01"/>
-      </geometry>
-      <material name="gray"/>
-    </visual>
-  </link>
-  <!-- Wheels -->
-  <xacro:wheel name="wheel_front_left" radius="${wheel_radius}" width="${wheel_width}"/>
-  <xacro:wheel name="wheel_front_right" radius="${wheel_radius}" width="${wheel_width}"/>
-  <xacro:wheel name="wheel_back_left" radius="${wheel_radius}" width="${wheel_width}"/>
-  <xacro:wheel name="wheel_back_right" radius="${wheel_radius}" width="${wheel_width}"/>
+  <xacro:fixed_joint name="joint_base_footprint" parent="base_footprint" child="base_link" origin_xyz="0 0 ${base_height / 2}" origin_rpy="0 0 0"/>
+  <!-- Base Axes -->
+  <xacro:base_axis name="base_axis_front_left" length="${base_axis_length}" radius="${base_axis_radius}"/>
+  <xacro:base_axis name="base_axis_front_right" length="${base_axis_length}" radius="${base_axis_radius}"/>
+  <xacro:base_axis name="base_axis_back_left" length="${base_axis_length}" radius="${base_axis_radius}"/>
+  <xacro:base_axis name="base_axis_back_right" length="${base_axis_length}" radius="${base_axis_radius}"/>
+  <!-- Base Axes Joints -->
+  <xacro:fixed_joint name="joint_base_axis_front_left" parent="base_link" child="base_axis_front_left" origin_xyz="${-base_width / 2} ${base_length / 2} 0" origin_rpy="0 ${pi/2} 0"/>
+  <xacro:fixed_joint name="joint_base_axis_front_right" parent="base_link" child="base_axis_front_right" origin_xyz="${base_width / 2} ${base_length / 2} 0" origin_rpy="0 ${pi/2} 0"/>
+  <xacro:fixed_joint name="joint_base_axis_back_left" parent="base_link" child="base_axis_back_left" origin_xyz="${-base_width / 2} ${-base_length / 2} 0" origin_rpy="0 ${pi/2} 0"/>
+  <xacro:fixed_joint name="joint_base_axis_back_right" parent="base_link" child="base_axis_back_right" origin_xyz="${base_width / 2} ${-base_length / 2} 0" origin_rpy="0 ${pi/2} 0"/>
   <!-- Motors -->
   <xacro:motor name="motor_front_left" length="${motor_length}" radius="${motor_radius}" mass="1.0" ixx="0.01" ixy="0.0" ixz="0.0" iyy="0.01" iyz="0.0" izz="0.01"/>
@@ -37,18 +37,21 @@
   <xacro:motor name="motor_back_right" length="${motor_length}" radius="${motor_radius}" mass="1.0" ixx="0.01" ixy="0.0" ixz="0.0" iyy="0.01" iyz="0.0" izz="0.01"/>
   <!-- Motor Joints -->
-  <xacro:fixed_joint name="joint_motor_front_left" parent="base_link" child="motor_front_left" origin_xyz="${-base_width / 2} ${base_length / 2} 0"/>
-  <xacro:fixed_joint name="joint_motor_front_right" parent="base_link" child="motor_front_right" origin_xyz="${base_width / 2} ${base_length / 2} 0"/>
-  <xacro:fixed_joint name="joint_motor_back_left" parent="base_link" child="motor_back_left" origin_xyz="${-base_width / 2} ${-base_length / 2} 0"/>
-  <xacro:fixed_joint name="joint_motor_back_right" parent="base_link" child="motor_back_right" origin_xyz="${base_width / 2} ${-base_length / 2} 0"/>
+  <xacro:fixed_joint name="joint_motor_front_left" parent="base_axis_front_left" child="motor_front_left" origin_xyz="0 0 0" origin_rpy="0 0 0"/>
+  <xacro:fixed_joint name="joint_motor_front_right" parent="base_axis_front_right" child="motor_front_right" origin_xyz="0 0 0" origin_rpy="0 0 0"/>
+  <xacro:fixed_joint name="joint_motor_back_left" parent="base_axis_back_left" child="motor_back_left" origin_xyz="0 0 0" origin_rpy="0 0 0"/>
+  <xacro:fixed_joint name="joint_motor_back_right" parent="base_axis_back_right" child="motor_back_right" origin_xyz="0 0 0" origin_rpy="0 0 0"/>
+  <!-- Wheels -->
+  <xacro:wheel name="wheel_front_left" radius="${wheel_radius}" width="${wheel_width}"/>
+  <xacro:wheel name="wheel_front_right" radius="${wheel_radius}" width="${wheel_width}"/>
+  <xacro:wheel name="wheel_back_left" radius="${wheel_radius}" width="${wheel_width}"/>
+  <xacro:wheel name="wheel_back_right" radius="${wheel_radius}" width="${wheel_width}"/>
   <!-- Wheels Joints -->
-  <xacro:fixed_joint name="joint_wheel_front_left" parent="motor_front_left" child="wheel_front_left" origin_xyz="0 0 ${wheel_radius}"/>
-  <xacro:fixed_joint name="joint_wheel_front_right" parent="motor_front_right" child="wheel_front_right" origin_xyz="0 0 ${wheel_radius}"/>
-  <xacro:fixed_joint name="joint_wheel_back_left" parent="motor_back_left" child="wheel_back_left" origin_xyz="0 0 ${wheel_radius}"/>
-  <xacro:fixed_joint name="joint_wheel_back_right" parent="motor_back_right" child="wheel_back_right" origin_xyz="0 0 ${wheel_radius}"/>
+  <xacro:fixed_joint name="joint_wheel_front_left" parent="base_axis_front_left" child="wheel_front_left" origin_xyz="0 0 -${motor_length/2}" origin_rpy="0 0 0"/>
+  <xacro:fixed_joint name="joint_wheel_front_right" parent="base_axis_front_right" child="wheel_front_right" origin_xyz="0 0 ${motor_length/2}" origin_rpy="0 0 0"/>
+  <xacro:fixed_joint name="joint_wheel_back_left" parent="base_axis_back_left" child="wheel_back_left" origin_xyz="0 0 -${motor_length/2}" origin_rpy="0 0 0"/>
+  <xacro:fixed_joint name="joint_wheel_back_right" parent="base_axis_back_right" child="wheel_back_right" origin_xyz="0 0 ${motor_length/2}" origin_rpy="0 0 0"/>
   <!-- Camera -->
   <xacro:camera name="camera" width="${camera_width}" length="${camera_length}" height="${camera_height}" radius="${camera_lens_radius}"/>
   <!-- Camera Joint -->
-  <xacro:fixed_joint name="joint_camera" parent="base_link" child="camera" origin_xyz="0 0 ${base_height}"/>
-  <!-- Base Footprint Joint -->
-  <xacro:fixed_joint name="joint_base_footprint" parent="base_link" child="base_footprint" origin_xyz="0 0 -${base_height / 2}"/>
+  <xacro:fixed_joint name="joint_camera" parent="base_link" child="camera" origin_xyz="0 0 ${base_height}" origin_rpy="0 0 0"/>
 </robot>

File: urdf/wheel.xacro (robot description, xacro)
@@ -7,5 +7,5 @@
           <cylinder length="${width}" radius="${radius}"/>
         </geometry>
-        <material name="black"/>
+        <material name="metallic_dark_lead"/>
       </visual>
       <collision>

Commit message: added joint_state_publisher to revolute joints.

File: urdf/base_axis.xacro (robot description, xacro)
@@ -7,4 +7,5 @@
           <cylinder length="${length}" radius="${radius}"/>
         </geometry>
+        <origin xyz="0 0 0" rpy="0 0 ${pi / 2.0}" />
         <material name="dark_red"/>
       </visual>
@@ -13,4 +14,5 @@
           <cylinder length="${length}" radius="${radius}"/>
         </geometry>
+        <origin xyz="0 0 0" rpy="0 0 ${pi / 2.0}" />
       </collision>
     </link>

File: urdf/shelfbot.urdf.xacro (robot description, xacro)
@@ -29,25 +29,4 @@
   <xacro:base_axis name="base_axis_back_left" length="${base_axis_length}" radius="${base_axis_radius}"/>
   <xacro:base_axis name="base_axis_back_right" length="${base_axis_length}" radius="${base_axis_radius}"/>
-  <!-- Base Axes Joints -->
-  <joint name="joint_base_axis_front_left" type="fixed">
-    <parent link="base_link"/>
-    <child link="base_axis_front_left"/>
-    <origin xyz="${-base_width / 2} ${base_length / 2} 0" rpy="0 ${pi/2} 0"/>
-  </joint>
-  <joint name="joint_base_axis_front_right" type="fixed">
-    <parent link="base_link"/>
-    <child link="base_axis_front_right"/>
-    <origin xyz="${base_width / 2} ${base_length / 2} 0" rpy="0 ${pi/2} 0"/>
-  </joint>
-  <joint name="joint_base_axis_back_left" type="fixed">
-    <parent link="base_link"/>
-    <child link="base_axis_back_left"/>
-    <origin xyz="${-base_width / 2} ${-base_length / 2} 0" rpy="0 ${pi/2} 0"/>
-  </joint>
-  <joint name="joint_base_axis_back_right" type="fixed">
-    <parent link="base_link"/>
-    <child link="base_axis_back_right"/>
-    <origin xyz="${base_width / 2} ${-base_length / 2} 0" rpy="0 ${pi/2} 0"/>
-  </joint>
   <!-- Motors -->
   <xacro:motor name="motor_front_left" length="${motor_length}" radius="${motor_radius}" mass="1.0" ixx="0.01" ixy="0.0" ixz="0.0" iyy="0.01" iyz="0.0" izz="0.01"/>
@@ -55,25 +34,4 @@
   <xacro:motor name="motor_back_left" length="${motor_length}" radius="${motor_radius}" mass="1.0" ixx="0.01" ixy="0.0" ixz="0.0" iyy="0.01" iyz="0.0" izz="0.01"/>
   <xacro:motor name="motor_back_right" length="${motor_length}" radius="${motor_radius}" mass="1.0" ixx="0.01" ixy="0.0" ixz="0.0" iyy="0.01" iyz="0.0" izz="0.01"/>
-  <!-- Motor Joints -->
-  <joint name="joint_motor_front_left" type="fixed">
-    <parent link="base_axis_front_left"/>
-    <child link="motor_front_left"/>
-    <origin xyz="0 0 0" rpy="0 0 0"/>
-  </joint>
-  <joint name="joint_motor_front_right" type="fixed">
-    <parent link="base_axis_front_right"/>
-    <child link="motor_front_right"/>
-    <origin xyz="0 0 0" rpy="0 0 0"/>
-  </joint>
-  <joint name="joint_motor_back_left" type="fixed">
-    <parent link="base_axis_back_left"/>
-    <child link="motor_back_left"/>
-    <origin xyz="0 0 0" rpy="0 0 0"/>
-  </joint>
-  <joint name="joint_motor_back_right" type="fixed">
-    <parent link="base_axis_back_right"/>
-    <child link="motor_back_right"/>
-    <origin xyz="0 0 0" rpy="0 0 0"/>
-  </joint>
   <!-- Wheels -->
   <xacro:wheel name="wheel_front_left" radius="${wheel_radius}" width="${wheel_width}"/>
@@ -81,4 +39,58 @@
   <xacro:wheel name="wheel_back_left" radius="${wheel_radius}" width="${wheel_width}"/>
   <xacro:wheel name="wheel_back_right" radius="${wheel_radius}" width="${wheel_width}"/>
+  <!-- Motor Joints -->
+  <joint name="joint_motor_front_left" type="fixed">
+    <parent link="base_link"/>
+    <child link="motor_front_left"/>
+    <origin xyz="${-base_width / 2} ${base_length / 2} 0" rpy="0 ${pi/2} 0"/>
+  </joint>
+  <joint name="joint_motor_front_right" type="fixed">
+    <parent link="base_link"/>
+    <child link="motor_front_right"/>
+    <origin xyz="${base_width / 2} ${base_length / 2} 0" rpy="0 ${pi/2} 0"/>
+  </joint>
+  <joint name="joint_motor_back_left" type="fixed">
+    <parent link="base_link"/>
+    <child link="motor_back_left"/>
+    <origin xyz="${-base_width / 2} ${-base_length / 2} 0" rpy="0 ${pi/2} 0"/>
+  </joint>
+  <joint name="joint_motor_back_right" type="fixed">
+    <parent link="base_link"/>
+    <child link="motor_back_right"/>
+    <origin xyz="${base_width / 2} ${-base_length / 2} 0" rpy="0 ${pi/2} 0"/>
+  </joint>
+  <!-- Base Axes Joints -->
+  <joint name="joint_base_axis_front_left" type="revolute">
+    <parent link="motor_front_left"/>
+    <child link="base_axis_front_left"/>
+    <origin xyz="0 0 0" rpy="0 0 0"/>
+    <axis xyz="0 1 0"/>
+    <limit lower="-3.14159" upper="3.14159" effort="100" velocity="1.0"/>
+    <dynamics damping="0.1" friction="0.1"/>
+  </joint>
+  <joint name="joint_base_axis_front_right" type="revolute">
+    <parent link="motor_front_right"/>
+    <child link="base_axis_front_right"/>
+    <origin xyz="0 0 0" rpy="0 0 0"/>
+    <axis xyz="0 1 0"/>
+    <limit lower="-3.14159" upper="3.14159" effort="100" velocity="1.0"/>
+    <dynamics damping="0.1" friction="0.1"/>
+  </joint>
+  <joint name="joint_base_axis_back_left" type="revolute">
+    <parent link="motor_back_left"/>
+    <child link="base_axis_back_left"/>
+    <origin xyz="0 0 0" rpy="0 0 0"/>
+    <axis xyz="0 1 0"/>
+    <limit lower="-3.14159" upper="3.14159" effort="100" velocity="1.0"/>
+    <dynamics damping="0.1" friction="0.1"/>
+  </joint>
+  <joint name="joint_base_axis_back_right" type="revolute">
+    <parent link="motor_back_right"/>
+    <child link="base_axis_back_right"/>
+    <origin xyz="0 0 0" rpy="0 0 0"/>
+    <axis xyz="0 1 0"/>
+    <limit lower="-3.14159" upper="3.14159" effort="100" velocity="1.0"/>
+    <dynamics damping="0.1" friction="0.1"/>
+  </joint>
   <!-- Wheels Joints -->
   <joint name="joint_wheel_front_left" type="fixed">
