Commit message: Adding inertia, drag and friction parameters,

File: urdf/base_axis.xacro (robot description, xacro)
@@ -16,4 +16,9 @@
         <origin xyz="0 0 0" rpy="0 0 ${pi / 2.0}" />
       </collision>
+      <inertial>
+        <mass value="${base_axis_mass}"/>
+        <origin xyz="0 0 0" rpy="0 0 ${pi / 2.0}"/>
+        <xacro:cylinder_inertia m="${base_axis_mass}" r="${radius}" h="${length}"/>
+      </inertial>
     </link>
   </xacro:macro>

File: urdf/camera.xacro (robot description, xacro)
@@ -7,5 +7,4 @@
         <geometry>
           <box size="${width} ${length} ${height}"/>
-          <cylinder length="0.05" radius="${radius}"/>
         </geometry>
         <material name="metallic_gray"/>
@@ -15,7 +14,11 @@
         <geometry>
           <box size="${width} ${length} ${height}"/>
-          <cylinder length="0.05" radius="${radius}"/>
         </geometry>
       </collision>
+      <inertial>
+        <mass value="${camera_mass}"/>
+        <origin xyz="0 0 ${height/2}" rpy="0 0 0"/>
+        <xacro:box_inertia m="${camera_mass}" x="${width}" y="${length}" z="${height}"/>
+      </inertial>
     </link>
   </xacro:macro>

File: urdf/common_properties.xacro (robot description, xacro)
@@ -16,8 +16,11 @@
   <xacro:property name="base_length" value="0.7"/>
   <xacro:property name="base_height" value="0.2"/>
+  <xacro:property name="base_mass" value="20.0"/>
   <xacro:property name="motor_radius" value="0.05"/>
   <xacro:property name="motor_length" value="0.2"/>
+  <xacro:property name="motor_mass" value="2.0"/>
   <xacro:property name="wheel_radius" value="0.2"/>
   <xacro:property name="wheel_width" value="0.05"/>
+  <xacro:property name="wheel_mass" value="3.0"/>
   <xacro:property name="camera_width" value="0.2"/>
   <xacro:property name="camera_length" value="0.2"/>
@@ -25,5 +28,17 @@
   <xacro:property name="camera_lens_radius" value="0.05"/>
   <xacro:property name="camera_mount_height" value="0.5"/>
+  <xacro:property name="camera_mass" value="0.5"/>
   <xacro:property name="base_axis_radius" value="0.02"/>
   <xacro:property name="base_axis_length" value="${motor_length + wheel_width}"/>
+  <xacro:property name="base_axis_mass" value="1.0"/>
+  <xacro:macro name="cylinder_inertia" params="m r h">
+    <inertia ixx="${m*(3*r*r+h*h)/12}" ixy="0" ixz="0"
+             iyy="${m*(3*r*r+h*h)/12}" iyz="0"
+             izz="${m*r*r/2}"/>
+  </xacro:macro>
+  <xacro:macro name="box_inertia" params="m x y z">
+    <inertia ixx="${m*(y*y+z*z)/12}" ixy="0" ixz="0"
+             iyy="${m*(x*x+z*z)/12}" iyz="0"
+             izz="${m*(x*x+y*y)/12}"/>
+  </xacro:macro>
 </robot>

File: urdf/gazebo.urdf.xacro (robot description, xacro)
@@ -4,65 +4,42 @@
     <material>Gazebo/Gold</material>
   </gazebo>
-  <gazebo reference="wheel_front_left">
-    <material>Gazebo/Black</material>
-  </gazebo>
-  <gazebo reference="wheel_front_right">
-    <material>Gazebo/Black</material>
-  </gazebo>
-  <gazebo reference="wheel_back_left">
-    <material>Gazebo/Black</material>
-  </gazebo>
-  <gazebo reference="wheel_back_right">
-    <material>Gazebo/Black</material>
-  </gazebo>
-  <gazebo reference="base_axis_front_left">
-    <material>Gazebo/Red</material>
-  </gazebo>
-  <gazebo reference="base_axis_front_right">
-    <material>Gazebo/Red</material>
-  </gazebo>
-  <gazebo reference="base_axis_back_left">
-    <material>Gazebo/Red</material>
-  </gazebo>
-  <gazebo reference="base_axis_back_right">
-    <material>Gazebo/Red</material>
-  </gazebo>
-  <gazebo reference="motor_front_left">
-    <material>Gazebo/Grey</material>
-  </gazebo>
-  <gazebo reference="motor_front_right">
-    <material>Gazebo/Grey</material>
-  </gazebo>
-  <gazebo reference="motor_back_left">
-    <material>Gazebo/Grey</material>
-  </gazebo>
-  <gazebo reference="motor_back_right">
-    <material>Gazebo/Grey</material>
-  </gazebo>
+  <xacro:macro name="wheel_gazebo" params="name">
+    <gazebo reference="${name}">
+      <material>Gazebo/Black</material>
+      <mu1>0.8</mu1>
+      <mu2>0.8</mu2>
+      <kp>1000000.0</kp>
+      <kd>100.0</kd>
+      <minDepth>0.001</minDepth>
+      <maxVel>1.0</maxVel>
+      <fdir1>1 0 0</fdir1>
+      <slip1>0.05</slip1>
+      <slip2>0.05</slip2>
+    </gazebo>
+  </xacro:macro>
+  <xacro:wheel_gazebo name="wheel_front_left"/>
+  <xacro:wheel_gazebo name="wheel_front_right"/>
+  <xacro:wheel_gazebo name="wheel_back_left"/>
+  <xacro:wheel_gazebo name="wheel_back_right"/>
+  <xacro:macro name="base_axis_gazebo" params="name">
+    <gazebo reference="${name}">
+      <material>Gazebo/Red</material>
+    </gazebo>
+  </xacro:macro>
+  <xacro:base_axis_gazebo name="base_axis_front_left"/>
+  <xacro:base_axis_gazebo name="base_axis_front_right"/>
+  <xacro:base_axis_gazebo name="base_axis_back_left"/>
+  <xacro:base_axis_gazebo name="base_axis_back_right"/>
+  <xacro:macro name="motor_gazebo" params="name">
+    <gazebo reference="${name}">
+      <material>Gazebo/Grey</material>
+    </gazebo>
+  </xacro:macro>
+  <xacro:motor_gazebo name="motor_front_left"/>
+  <xacro:motor_gazebo name="motor_front_right"/>
+  <xacro:motor_gazebo name="motor_back_left"/>
+  <xacro:motor_gazebo name="motor_back_right"/>
   <gazebo reference="camera">
     <material>Gazebo/Blue</material>
-  </gazebo>
-  <gazebo reference="joint_base_axis_front_left">
-    <provideFeedback>true</provideFeedback>
-    <implicitSpringDamper>true</implicitSpringDamper>
-  </gazebo>
-  <gazebo reference="joint_base_axis_front_right">
-    <provideFeedback>true</provideFeedback>
-    <implicitSpringDamper>true</implicitSpringDamper>
-  </gazebo>
-  <gazebo reference="joint_base_axis_back_left">
-    <provideFeedback>true</provideFeedback>
-    <implicitSpringDamper>true</implicitSpringDamper>
-  </gazebo>
-  <gazebo reference="joint_base_axis_back_right">
-    <provideFeedback>true</provideFeedback>
-    <implicitSpringDamper>true</implicitSpringDamper>
-  </gazebo>
-  <gazebo>
-    <plugin name="gazebo_ros2_control" filename="libgazebo_ros2_control.so">
-      <parameters>$(find shelfbot)/config/four_wheel_drive_controller.yaml</parameters>
-    </plugin>
-  </gazebo>
-  <gazebo reference="camera">
     <sensor type="camera" name="camera">
       <update_rate>30.0</update_rate>
@@ -89,3 +66,18 @@
     </sensor>
   </gazebo>
+  <xacro:macro name="base_axis_joint_gazebo" params="name">
+    <gazebo reference="${name}">
+      <provideFeedback>true</provideFeedback>
+      <implicitSpringDamper>true</implicitSpringDamper>
+    </gazebo>
+  </xacro:macro>
+  <xacro:base_axis_joint_gazebo name="joint_base_axis_front_left"/>
+  <xacro:base_axis_joint_gazebo name="joint_base_axis_front_right"/>
+  <xacro:base_axis_joint_gazebo name="joint_base_axis_back_left"/>
+  <xacro:base_axis_joint_gazebo name="joint_base_axis_back_right"/>
+  <gazebo>
+    <plugin name="gazebo_ros2_control" filename="libgazebo_ros2_control.so">
+      <parameters>$(find shelfbot)/config/four_wheel_drive_controller.yaml</parameters>
+    </plugin>
+  </gazebo>
 </robot>

File: urdf/motor.xacro (robot description, xacro)
@@ -1,5 +1,5 @@
 <?xml version="1.0"?>
 <robot xmlns:xacro="http://www.ros.org/wiki/xacro">
-  <xacro:macro name="motor" params="name length radius mass ixx ixy ixz iyy iyz izz">
+  <xacro:macro name="motor" params="name length radius">
     <link name="${name}">
       <visual>
@@ -15,7 +15,7 @@
       </collision>
       <inertial>
-        <mass value="${mass}"/>
+        <mass value="${motor_mass}"/>
         <origin xyz="0 0 0" rpy="0 0 0"/>
-        <inertia ixx="${ixx}" ixy="${ixy}" ixz="${ixz}" iyy="${iyy}" iyz="${iyz}" izz="${izz}"/>
+        <xacro:cylinder_inertia m="${motor_mass}" r="${radius}" h="${length}"/>
       </inertial>
     </link>

File: urdf/shelfbot.urdf.xacro (robot description, xacro)
@@ -21,6 +21,7 @@
     </collision>
     <inertial>
-      <mass value="5"/>
-      <inertia ixx="0.0395" ixy="0" ixz="0" iyy="0.086" iyz="0" izz="0.0754"/>
+      <mass value="${base_mass}"/>
+      <origin xyz="0 0 0" rpy="0 0 0"/>
+      <xacro:box_inertia m="${base_mass}" x="${base_width}" y="${base_length}" z="${base_height}"/>
     </inertial>
   </link>
@@ -34,8 +35,8 @@
   <xacro:base_axis name="base_axis_back_left" length="${base_axis_length}" radius="${base_axis_radius}"/>
   <xacro:base_axis name="base_axis_back_right" length="${base_axis_length}" radius="${base_axis_radius}"/>
-  <xacro:motor name="motor_front_left" length="${motor_length}" radius="${motor_radius}" mass="1.0" ixx="0.01" ixy="0.0" ixz="0.0" iyy="0.01" iyz="0.0" izz="0.01"/>
-  <xacro:motor name="motor_front_right" length="${motor_length}" radius="${motor_radius}" mass="1.0" ixx="0.01" ixy="0.0" ixz="0.0" iyy="0.01" iyz="0.0" izz="0.01"/>
-  <xacro:motor name="motor_back_left" length="${motor_length}" radius="${motor_radius}" mass="1.0" ixx="0.01" ixy="0.0" ixz="0.0" iyy="0.01" iyz="0.0" izz="0.01"/>
-  <xacro:motor name="motor_back_right" length="${motor_length}" radius="${motor_radius}" mass="1.0" ixx="0.01" ixy="0.0" ixz="0.0" iyy="0.01" iyz="0.0" izz="0.01"/>
+  <xacro:motor name="motor_front_left" length="${motor_length}" radius="${motor_radius}"/>
+  <xacro:motor name="motor_front_right" length="${motor_length}" radius="${motor_radius}"/>
+  <xacro:motor name="motor_back_left" length="${motor_length}" radius="${motor_radius}"/>
+  <xacro:motor name="motor_back_right" length="${motor_length}" radius="${motor_radius}"/>
   <xacro:wheel name="wheel_front_left" radius="${wheel_radius}" width="${wheel_width}"/>
   <xacro:wheel name="wheel_front_right" radius="${wheel_radius}" width="${wheel_width}"/>
@@ -67,5 +68,5 @@
     <origin xyz="0 0 0" rpy="0 0 0"/>
     <axis xyz="0 0 1"/>
-    <limit effort="10" velocity="10"/>
+    <dynamics damping="0.1" friction="0.1"/>
   </joint>
   <joint name="joint_base_axis_front_right" type="continuous">
@@ -74,5 +75,5 @@
     <origin xyz="0 0 0" rpy="0 0 0"/>
     <axis xyz="0 0 1"/>
-    <limit effort="10" velocity="10"/>
+    <dynamics damping="0.1" friction="0.1"/>
   </joint>
   <joint name="joint_base_axis_back_left" type="continuous">
@@ -81,5 +82,5 @@
     <origin xyz="0 0 0" rpy="0 0 0"/>
     <axis xyz="0 0 1"/>
-    <limit effort="10" velocity="10"/>
+    <dynamics damping="0.1" friction="0.1"/>
   </joint>
   <joint name="joint_base_axis_back_right" type="continuous">
@@ -88,5 +89,5 @@
     <origin xyz="0 0 0" rpy="0 0 0"/>
     <axis xyz="0 0 1"/>
-    <limit effort="10" velocity="10"/>
+    <dynamics damping="0.1" friction="0.1"/>
   </joint>
   <joint name="joint_wheel_front_left" type="fixed">

File: urdf/wheel.xacro (robot description, xacro)
@@ -15,7 +15,7 @@
       </collision>
       <inertial>
-        <mass value="0.5"/>
+        <mass value="${wheel_mass}"/>
         <origin xyz="0 0 0" rpy="0 0 0"/>
-        <inertia ixx="0.005" ixy="0.0" ixz="0.0" iyy="0.005" iyz="0.0" izz="0.005"/>
+        <xacro:cylinder_inertia m="${wheel_mass}" r="${radius}" h="${width}"/>
       </inertial>
     </link>

Commit message: Changing the rotation axis from z to x in elements, adjusting everything else around.

File: urdf/base_axis.xacro (robot description, xacro)
@@ -7,5 +7,5 @@
           <cylinder length="${length}" radius="${radius}"/>
         </geometry>
-        <origin xyz="0 0 0" rpy="0 0 ${pi / 2.0}" />
+        <origin xyz="${length/2} 0 0" rpy="0 ${pi/2} 0"/>
         <material name="dark_red"/>
       </visual>
@@ -14,9 +14,9 @@
           <cylinder length="${length}" radius="${radius}"/>
         </geometry>
-        <origin xyz="0 0 0" rpy="0 0 ${pi / 2.0}" />
+        <origin xyz="${length/2} 0 0" rpy="0 ${pi/2} 0"/>
       </collision>
       <inertial>
         <mass value="${base_axis_mass}"/>
-        <origin xyz="0 0 0" rpy="0 0 ${pi / 2.0}"/>
+        <origin xyz="${length/2} 0 0" rpy="0 ${pi/2} 0"/>
         <xacro:cylinder_inertia m="${base_axis_mass}" r="${radius}" h="${length}"/>
       </inertial>

File: urdf/gazebo.urdf.xacro (robot description, xacro)
@@ -70,4 +70,5 @@
           <far>300</far>
         </clip>
+        <pose>0 0 0 0 ${pi/2} 0</pose>
       </camera>
       <plugin name="camera_controller" filename="libgazebo_ros_camera.so">
@@ -91,4 +92,20 @@
   <xacro:base_axis_joint_gazebo name="joint_base_axis_back_left"/>
   <xacro:base_axis_joint_gazebo name="joint_base_axis_back_right"/>
+  <xacro:macro name="wheel_transmission" params="name">
+    <transmission name="${name}_transmission">
+      <type>transmission_interface/SimpleTransmission</type>
+      <joint name="${name}">
+        <hardwareInterface>hardware_interface/PositionJointInterface</hardwareInterface>
+      </joint>
+      <actuator name="${name}_motor">
+        <hardwareInterface>hardware_interface/PositionJointInterface</hardwareInterface>
+        <mechanicalReduction>1</mechanicalReduction>
+      </actuator>
+    </transmission>
+  </xacro:macro>
+  <xacro:wheel_transmission name="joint_wheel_front_left"/>
+  <xacro:wheel_transmission name="joint_wheel_front_right"/>
+  <xacro:wheel_transmission name="joint_wheel_back_left"/>
+  <xacro:wheel_transmission name="joint_wheel_back_right"/>
   <gazebo>
     <plugin name="gazebo_ros2_control" filename="libgazebo_ros2_control.so">

File: urdf/motor.xacro (robot description, xacro)
@@ -7,4 +7,5 @@
           <cylinder length="${length}" radius="${radius}"/>
         </geometry>
+        <origin xyz="${length/2} 0 0" rpy="0 ${pi/2} 0"/>
         <material name="metallic_gray"/>
       </visual>
@@ -13,8 +14,9 @@
           <cylinder length="${length}" radius="${radius}"/>
         </geometry>
+        <origin xyz="${length/2} 0 0" rpy="0 ${pi/2} 0"/>
       </collision>
       <inertial>
         <mass value="${motor_mass}"/>
-        <origin xyz="0 0 0" rpy="0 0 0"/>
+        <origin xyz="${length/2} 0 0" rpy="0 ${pi/2} 0"/>
         <xacro:cylinder_inertia m="${motor_mass}" r="${radius}" h="${length}"/>
       </inertial>

File: urdf/shelfbot.urdf.xacro (robot description, xacro)
@@ -46,26 +46,26 @@
     <parent link="base_link"/>
     <child link="motor_front_left"/>
-    <origin xyz="${-base_width / 2} ${base_length / 2} 0" rpy="0 ${pi/2} 0"/>
+    <origin xyz="${-base_width / 2 + motor_length / 2} ${base_length / 2} 0" rpy="${pi/2} 0 ${pi}"/>
   </joint>
   <joint name="joint_motor_front_right" type="fixed">
     <parent link="base_link"/>
     <child link="motor_front_right"/>
-    <origin xyz="${base_width / 2} ${base_length / 2} 0" rpy="0 ${pi/2} 0"/>
+    <origin xyz="${base_width / 2 - motor_length / 2} ${base_length / 2} 0" rpy="${-pi/2} 0 0"/>
   </joint>
   <joint name="joint_motor_back_left" type="fixed">
     <parent link="base_link"/>
     <child link="motor_back_left"/>
-    <origin xyz="${-base_width / 2} ${-base_length / 2} 0" rpy="0 ${pi/2} 0"/>
+    <origin xyz="${-base_width / 2 + motor_length / 2} ${-base_length / 2} 0" rpy="${pi/2} 0 ${pi}"/>
   </joint>
   <joint name="joint_motor_back_right" type="fixed">
     <parent link="base_link"/>
     <child link="motor_back_right"/>
-    <origin xyz="${base_width / 2} ${-base_length / 2} 0" rpy="0 ${pi/2} 0"/>
+    <origin xyz="${base_width / 2 - motor_length / 2} ${-base_length / 2} 0" rpy="${-pi/2} 0 0"/>
   </joint>
   <joint name="joint_base_axis_front_left" type="continuous">
     <parent link="motor_front_left"/>
     <child link="base_axis_front_left"/>
-    <origin xyz="0 0 0" rpy="0 0 0"/>
-    <axis xyz="0 0 1"/>
+    <origin xyz="${motor_length/2} 0 0" rpy="${-pi/2} 0 0"/>
+    <axis xyz="1 0 0"/>
     <dynamics damping="0.1" friction="0.1"/>
   </joint>
@@ -73,6 +73,6 @@
     <parent link="motor_front_right"/>
     <child link="base_axis_front_right"/>
-    <origin xyz="0 0 0" rpy="0 0 0"/>
-    <axis xyz="0 0 1"/>
+    <origin xyz="${motor_length/2} 0 0" rpy="${pi/2} 0 0"/>
+    <axis xyz="1 0 0"/>
     <dynamics damping="0.1" friction="0.1"/>
   </joint>
@@ -80,6 +80,6 @@
     <parent link="motor_back_left"/>
     <child link="base_axis_back_left"/>
-    <origin xyz="0 0 0" rpy="0 0 0"/>
-    <axis xyz="0 0 1"/>
+    <origin xyz="${motor_length/2} 0 0" rpy="${-pi/2} 0 0"/>
+    <axis xyz="1 0 0"/>
     <dynamics damping="0.1" friction="0.1"/>
   </joint>
@@ -87,6 +87,6 @@
     <parent link="motor_back_right"/>
     <child link="base_axis_back_right"/>
-    <origin xyz="0 0 0" rpy="0 0 0"/>
-    <axis xyz="0 0 1"/>
+    <origin xyz="${motor_length/2} 0 0" rpy="${pi/2} 0 0"/>
+    <axis xyz="1 0 0"/>
     <dynamics damping="0.1" friction="0.1"/>
   </joint>
@@ -94,6 +94,6 @@
     <parent link="base_axis_front_left"/>
     <child link="wheel_front_left"/>
-    <origin xyz="0 0 -${motor_length/2}" rpy="0 0 0"/>
-    <axis xyz="0 0 1"/>
+    <origin xyz="${base_axis_length - wheel_width} 0 0" rpy="0 0 0"/>
+    <axis xyz="1 0 0"/>
     <mimic joint="joint_base_axis_front_left" multiplier="${gear_ratio}" offset="0"/>
   </joint>
@@ -101,6 +101,6 @@
     <parent link="base_axis_front_right"/>
     <child link="wheel_front_right"/>
-    <origin xyz="0 0 ${motor_length/2}" rpy="0 0 0"/>
-    <axis xyz="0 0 1"/>
+    <origin xyz="${base_axis_length - wheel_width} 0 0" rpy="0 0 0"/>
+    <axis xyz="1 0 0"/>
     <mimic joint="joint_base_axis_front_right" multiplier="${gear_ratio}" offset="0"/>
   </joint>
@@ -108,6 +108,6 @@
     <parent link="base_axis_back_left"/>
     <child link="wheel_back_left"/>
-    <origin xyz="0 0 -${motor_length/2}" rpy="0 0 0"/>
-    <axis xyz="0 0 1"/>
+    <origin xyz="${base_axis_length - wheel_width} 0 0" rpy="0 0 0"/>
+    <axis xyz="1 0 0"/>
     <mimic joint="joint_base_axis_back_left" multiplier="${gear_ratio}" offset="0"/>
   </joint>
@@ -115,6 +115,6 @@
     <parent link="base_axis_back_right"/>
     <child link="wheel_back_right"/>
-    <origin xyz="0 0 ${motor_length/2}" rpy="0 0 0"/>
-    <axis xyz="0 0 1"/>
+    <origin xyz="${base_axis_length - wheel_width} 0 0" rpy="0 0 0"/>
+    <axis xyz="1 0 0"/>
     <mimic joint="joint_base_axis_back_right" multiplier="${gear_ratio}" offset="0"/>
   </joint>
@@ -123,5 +123,5 @@
     <parent link="base_link"/>
     <child link="camera"/>
-    <origin xyz="0 0 ${base_height}" rpy="0 0 0"/>
+    <origin xyz="0 0 ${base_height}" rpy="${-pi/2} 0 0"/>
   </joint>
   <ros2_control name="FourWheelDriveSystem" type="system">

File: urdf/wheel.xacro (robot description, xacro)
@@ -7,4 +7,5 @@
           <cylinder length="${width}" radius="${radius}"/>
         </geometry>
+        <origin xyz="${width/2} 0 0" rpy="0 ${pi/2} 0"/>
         <material name="metallic_dark_lead"/>
       </visual>
@@ -13,8 +14,9 @@
           <cylinder length="${width}" radius="${radius}"/>
         </geometry>
+        <origin xyz="${width/2} 0 0" rpy="0 ${pi/2} 0"/>
       </collision>
       <inertial>
         <mass value="${wheel_mass}"/>
-        <origin xyz="0 0 0" rpy="0 0 0"/>
+        <origin xyz="${width/2} 0 0" rpy="0 ${pi/2} 0"/>
         <xacro:cylinder_inertia m="${wheel_mass}" r="${radius}" h="${width}"/>
       </inertial>
