Commit message: feat(robot): Add ultrasonic sensors and enable closed-loop control
This commit introduces two major improvements to the robots configuration:

1.  **URDF:** Adds a 6-sensor ultrasonic array for obstacle avoidance.
    - Creates a new `ultrasonic_sensor.xacro` macro for the HC-SR04.
    - Instantiates 3 sensors on the front and 3 on the back of the robot for comprehensive coverage.
    - Refactors the URDF to define materials only once in `common_properties.xacro` to fix parsing errors.

2.  **Control:** Switches the `four_wheel_drive_controller` to closed-loop mode by setting `open_loop: false`. This uses motor feedback to significantly reduce jitter and improve movement smoothness.

File: urdf/base_axis.xacro (robot description, xacro)
@@ -8,5 +8,4 @@
         </geometry>
         <origin xyz="${length/2} 0 0" rpy="0 ${pi/2} 0"/>
-        <material name="dark_red"/>
       </visual>
       <collision>

File: urdf/box.xacro (robot description, xacro)
@@ -7,5 +7,4 @@
           <box size="0.05 0.05 0.1"/>
         </geometry>
-        <material name="red"/>
       </visual>
       <collision>

File: urdf/camera.xacro (robot description, xacro)
@@ -8,5 +8,4 @@
           <box size="${width} ${length} ${height}"/>
         </geometry>
-        <material name="metallic_gray"/>
       </visual>
       <collision>

File: urdf/common_properties.xacro (robot description, xacro)
@@ -17,4 +17,10 @@
   <material name="red">
     <color rgba="1.0 0.0 0.0 1.0"/>
+  </material>
+  <material name="blue">
+    <color rgba="0.0 0.0 1.0 1.0"/>
+  </material>
+  <material name="light_grey">
+    <color rgba="0.8 0.8 0.8 1.0"/>
   </material>
   <xacro:property name="base_width" value="${config['four_wheel_drive_controller']['ros__parameters']['base_width']}"/>

File: urdf/motor.xacro (robot description, xacro)
@@ -8,5 +8,4 @@
         </geometry>
         <origin xyz="${length/2} 0 0" rpy="0 ${pi/2} 0"/>
-        <material name="metallic_gray"/>
       </visual>
       <collision>

File: urdf/shelfbot.urdf.xacro (robot description, xacro)
@@ -8,4 +8,5 @@
   <xacro:include filename="$(find shelfbot)/urdf/base_axis.xacro"/>
   <xacro:include filename="$(find shelfbot)/urdf/box.xacro"/>
+  <xacro:include filename="$(find shelfbot)/urdf/ultrasonic_sensor.xacro"/>
   <!-- Declare the arguments that will be passed in from the launch file -->
   <xacro:arg name="sim_mode" default="gazebo"/>
@@ -137,3 +138,40 @@
     <origin xyz="0 0 ${base_height}" rpy="${-pi/2} 0 0"/>
   </joint>
+  <!-- Ultrasonic Sensors (3-Front, 3-Back Configuration) -->
+  <xacro:ultrasonic_sensor name="us_front_center"/>
+  <xacro:ultrasonic_sensor name="us_front_left_corner"/>
+  <xacro:ultrasonic_sensor name="us_front_right_corner"/>
+  <xacro:ultrasonic_sensor name="us_back_center"/>
+  <xacro:ultrasonic_sensor name="us_back_left_corner"/>
+  <xacro:ultrasonic_sensor name="us_back_right_corner"/>
+  <joint name="joint_us_front_center" type="fixed">
+    <parent link="base_link"/>
+    <child link="us_front_center"/>
+    <origin xyz="0 ${base_length / 2} 0.01" rpy="0 ${pi/2} ${pi/2}"/>
+  </joint>
+  <joint name="joint_us_front_left_corner" type="fixed">
+    <parent link="base_link"/>
+    <child link="us_front_left_corner"/>
+    <origin xyz="${base_width / 4} ${base_length / 2} 0.01" rpy="0 ${pi/2} ${pi/4}"/>
+  </joint>
+  <joint name="joint_us_front_right_corner" type="fixed">
+    <parent link="base_link"/>
+    <child link="us_front_right_corner"/>
+    <origin xyz="${-base_width / 4} ${base_length / 2} 0.01" rpy="0 ${pi/2} ${3*pi/4}"/>
+  </joint>
+  <joint name="joint_us_back_center" type="fixed">
+    <parent link="base_link"/>
+    <child link="us_back_center"/>
+    <origin xyz="0 ${-base_length / 2} 0.01" rpy="0 ${pi/2} ${-pi/2}"/>
+  </joint>
+  <joint name="joint_us_back_left_corner" type="fixed">
+    <parent link="base_link"/>
+    <child link="us_back_left_corner"/>
+    <origin xyz="${base_width / 4} ${-base_length / 2} 0.01" rpy="0 ${pi/2} ${-pi/4}"/>
+  </joint>
+  <joint name="joint_us_back_right_corner" type="fixed">
+    <parent link="base_link"/>
+    <child link="us_back_right_corner"/>
+    <origin xyz="${-base_width / 4} ${-base_length / 2} 0.01" rpy="0 ${pi/2} ${-3*pi/4}"/>
+  </joint>
 </robot>

File: urdf/wheel.xacro (robot description, xacro)
@@ -8,5 +8,4 @@
         </geometry>
         <origin xyz="${width/2} 0 0" rpy="0 ${pi/2} 0"/>
-        <material name="metallic_dark_lead"/>
       </visual>
       <collision>
