Commit message: Adding basic gazebo properties and gazebo world.

File: urdf/gazebo.urdf.xacro (robot description, xacro)
@@ -1,27 +1,35 @@
 <?xml version="1.0"?>
 <robot xmlns:xacro="http://www.ros.org/wiki/xacro">
-  <xacro:macro name="gazebo_properties" params="link">
+  <xacro:macro name="gazebo_link_properties" params="link color">
     <gazebo reference="${link}">
-      <material>Gazebo/Grey</material>
+      <material>Gazebo/${color}</material>
       <mu1>0.2</mu1>
       <mu2>0.2</mu2>
+      <kp>1000000.0</kp>
+      <kd>100.0</kd>
+      <maxVel>1.0</maxVel>
+      <minDepth>0.001</minDepth>
     </gazebo>
   </xacro:macro>
-  <xacro:macro name="wheel_gazebo" params="name">
-    <gazebo reference="${name}">
-      <material>Gazebo/Black</material>
-      <mu1>1.0</mu1>
-      <mu2>1.0</mu2>
-      <kp>1000000.0</kp>
-      <kd>100.0</kd>
-      <minDepth>0.001</minDepth>
-      <maxVel>1.0</maxVel>
-    </gazebo>
-  </xacro:macro>
+  <!-- Apply properties to links -->
+  <xacro:gazebo_link_properties link="base_link" color="Gold"/>
+  <xacro:gazebo_link_properties link="wheel_front_left" color="Black"/>
+  <xacro:gazebo_link_properties link="wheel_front_right" color="Black"/>
+  <xacro:gazebo_link_properties link="wheel_back_left" color="Black"/>
+  <xacro:gazebo_link_properties link="wheel_back_right" color="Black"/>
+  <xacro:gazebo_link_properties link="base_axis_front_left" color="Red"/>
+  <xacro:gazebo_link_properties link="base_axis_front_right" color="Red"/>
+  <xacro:gazebo_link_properties link="base_axis_back_left" color="Red"/>
+  <xacro:gazebo_link_properties link="base_axis_back_right" color="Red"/>
+  <xacro:gazebo_link_properties link="motor_front_left" color="Grey"/>
+  <xacro:gazebo_link_properties link="motor_front_right" color="Grey"/>
+  <xacro:gazebo_link_properties link="motor_back_left" color="Grey"/>
+  <xacro:gazebo_link_properties link="motor_back_right" color="Grey"/>
+  <xacro:gazebo_link_properties link="camera" color="Blue"/>
   <gazebo>
     <plugin name="differential_drive_controller" filename="libgazebo_ros_diff_drive.so">
       <updateRate>100.0</updateRate>
-      <leftJoint>front_left_wheel_joint</leftJoint>
-      <rightJoint>front_right_wheel_joint</rightJoint>
+      <leftJoint>joint_wheel_front_left</leftJoint>
+      <rightJoint>joint_wheel_front_right</rightJoint>
       <wheelSeparation>${base_width}</wheelSeparation>
       <wheelDiameter>${2*wheel_radius}</wheelDiameter>

Commit message: Adding a new driver for a four wheel robot.

File: urdf/gazebo.urdf.xacro (robot description, xacro)
@@ -1,42 +1,62 @@
 <?xml version="1.0"?>
 <robot xmlns:xacro="http://www.ros.org/wiki/xacro">
-  <xacro:macro name="gazebo_link_properties" params="link color">
-    <gazebo reference="${link}">
-      <material>Gazebo/${color}</material>
-      <mu1>0.2</mu1>
-      <mu2>0.2</mu2>
-      <kp>1000000.0</kp>
-      <kd>100.0</kd>
-      <maxVel>1.0</maxVel>
-      <minDepth>0.001</minDepth>
-    </gazebo>
-  </xacro:macro>
-  <!-- Apply properties to links -->
-  <xacro:gazebo_link_properties link="base_link" color="Gold"/>
-  <xacro:gazebo_link_properties link="wheel_front_left" color="Black"/>
-  <xacro:gazebo_link_properties link="wheel_front_right" color="Black"/>
-  <xacro:gazebo_link_properties link="wheel_back_left" color="Black"/>
-  <xacro:gazebo_link_properties link="wheel_back_right" color="Black"/>
-  <xacro:gazebo_link_properties link="base_axis_front_left" color="Red"/>
-  <xacro:gazebo_link_properties link="base_axis_front_right" color="Red"/>
-  <xacro:gazebo_link_properties link="base_axis_back_left" color="Red"/>
-  <xacro:gazebo_link_properties link="base_axis_back_right" color="Red"/>
-  <xacro:gazebo_link_properties link="motor_front_left" color="Grey"/>
-  <xacro:gazebo_link_properties link="motor_front_right" color="Grey"/>
-  <xacro:gazebo_link_properties link="motor_back_left" color="Grey"/>
-  <xacro:gazebo_link_properties link="motor_back_right" color="Grey"/>
-  <xacro:gazebo_link_properties link="camera" color="Blue"/>
+  <!-- Gazebo colors for each link -->
+  <gazebo reference="base_link">
+    <material>Gazebo/Gold</material>
+  </gazebo>
+  <gazebo reference="wheel_front_left">
+    <material>Gazebo/Black</material>
+  </gazebo>
+  <gazebo reference="wheel_front_right">
+    <material>Gazebo/Black</material>
+  </gazebo>
+  <gazebo reference="wheel_back_left">
+    <material>Gazebo/Black</material>
+  </gazebo>
+  <gazebo reference="wheel_back_right">
+    <material>Gazebo/Black</material>
+  </gazebo>
+  <gazebo reference="base_axis_front_left">
+    <material>Gazebo/Red</material>
+  </gazebo>
+  <gazebo reference="base_axis_front_right">
+    <material>Gazebo/Red</material>
+  </gazebo>
+  <gazebo reference="base_axis_back_left">
+    <material>Gazebo/Red</material>
+  </gazebo>
+  <gazebo reference="base_axis_back_right">
+    <material>Gazebo/Red</material>
+  </gazebo>
+  <gazebo reference="motor_front_left">
+    <material>Gazebo/Grey</material>
+  </gazebo>
+  <gazebo reference="motor_front_right">
+    <material>Gazebo/Grey</material>
+  </gazebo>
+  <gazebo reference="motor_back_left">
+    <material>Gazebo/Grey</material>
+  </gazebo>
+  <gazebo reference="motor_back_right">
+    <material>Gazebo/Grey</material>
+  </gazebo>
+  <gazebo reference="camera">
+    <material>Gazebo/Blue</material>
+  </gazebo>
+  <!-- Gazebo plugin for 4-wheeled robot control -->
   <gazebo>
-    <plugin name="differential_drive_controller" filename="libgazebo_ros_diff_drive.so">
+    <plugin name="skid_steer_drive_controller" filename="libgazebo_ros_skid_steer_drive.so">
       <updateRate>100.0</updateRate>
-      <leftJoint>joint_wheel_front_left</leftJoint>
-      <rightJoint>joint_wheel_front_right</rightJoint>
+      <robotNamespace>/</robotNamespace>
+      <leftFrontJoint>joint_base_axis_front_left</leftFrontJoint>
+      <rightFrontJoint>joint_base_axis_front_right</rightFrontJoint>
+      <leftRearJoint>joint_base_axis_back_left</leftRearJoint>
+      <rightRearJoint>joint_base_axis_back_right</rightRearJoint>
       <wheelSeparation>${base_width}</wheelSeparation>
       <wheelDiameter>${2*wheel_radius}</wheelDiameter>
       <robotBaseFrame>base_link</robotBaseFrame>
-      <publishWheelTF>true</publishWheelTF>
-      <publishOdomTF>true</publishOdomTF>
-      <publishWheelJointState>true</publishWheelJointState>
-      <odometrySource>world</odometrySource>
+      <torque>20</torque>
+      <topicName>cmd_vel</topicName>
+      <broadcastTF>true</broadcastTF>
     </plugin>
   </gazebo>

File: urdf/shelfbot.urdf.xacro (robot description, xacro)
@@ -7,4 +7,6 @@
   <xacro:include filename="$(find shelfbot)/urdf/camera.xacro"/>
   <xacro:include filename="$(find shelfbot)/urdf/base_axis.xacro"/>
+  <!-- Fix: Include the Gazebo-specific properties -->
+  <xacro:include filename="$(find shelfbot)/urdf/gazebo.urdf.xacro"/>
   <!-- Base Footprint Link -->
   <link name="base_footprint"/>
@@ -17,4 +19,13 @@
       <material name="golden_brown"/>
     </visual>
+    <collision>
+      <geometry>
+        <box size="${base_width} ${base_length} ${base_height}"/>
+      </geometry>
+    </collision>
+    <inertial>
+      <mass value="5"/>
+      <inertia ixx="0.0395" ixy="0" ixz="0" iyy="0.086" iyz="0" izz="0.0754"/>
+    </inertial>
   </link>
   <!-- Joint to raise base_link -->
@@ -61,35 +72,27 @@
   </joint>
   <!-- Base Axes Joints -->
-  <joint name="joint_base_axis_front_left" type="revolute">
+  <joint name="joint_base_axis_front_left" type="continuous">
     <parent link="motor_front_left"/>
     <child link="base_axis_front_left"/>
     <origin xyz="0 0 0" rpy="0 0 0"/>
     <axis xyz="0 0 1"/>
-    <limit lower="-3.14159" upper="3.14159" effort="100" velocity="1.0"/>
-    <dynamics damping="0.1" friction="0.1"/>
   </joint>
-  <joint name="joint_base_axis_front_right" type="revolute">
+  <joint name="joint_base_axis_front_right" type="continuous">
     <parent link="motor_front_right"/>
     <child link="base_axis_front_right"/>
     <origin xyz="0 0 0" rpy="0 0 0"/>
     <axis xyz="0 0 1"/>
-    <limit lower="-3.14159" upper="3.14159" effort="100" velocity="1.0"/>
-    <dynamics damping="0.1" friction="0.1"/>
   </joint>
-  <joint name="joint_base_axis_back_left" type="revolute">
+  <joint name="joint_base_axis_back_left" type="continuous">
     <parent link="motor_back_left"/>
     <child link="base_axis_back_left"/>
     <origin xyz="0 0 0" rpy="0 0 0"/>
     <axis xyz="0 0 1"/>
-    <limit lower="-3.14159" upper="3.14159" effort="100" velocity="1.0"/>
-    <dynamics damping="0.1" friction="0.1"/>
   </joint>
-  <joint name="joint_base_axis_back_right" type="revolute">
+  <joint name="joint_base_axis_back_right" type="continuous">
     <parent link="motor_back_right"/>
     <child link="base_axis_back_right"/>
     <origin xyz="0 0 0" rpy="0 0 0"/>
     <axis xyz="0 0 1"/>
-    <limit lower="-3.14159" upper="3.14159" effort="100" velocity="1.0"/>
-    <dynamics damping="0.1" friction="0.1"/>
   </joint>
   <!-- Wheels Joints -->

Commit message: Starting ros2_control custom plugin.

File: urdf/gazebo.urdf.xacro (robot description, xacro)
@@ -44,19 +44,8 @@
     <material>Gazebo/Blue</material>
   </gazebo>
-  <!-- Gazebo plugin for 4-wheeled robot control -->
+  <!-- Gazebo plugin for ros2_control -->
   <gazebo>
-    <plugin name="four_wheel_drive_controller" filename="libgazebo_ros_four_wheel_drive.so">
-      <updateRate>100.0</updateRate>
-      <robotNamespace>/</robotNamespace>
-      <leftFrontJoint>joint_base_axis_front_left</leftFrontJoint>
-      <rightFrontJoint>joint_base_axis_front_right</rightFrontJoint>
-      <leftRearJoint>joint_base_axis_back_left</leftRearJoint>
-      <rightRearJoint>joint_base_axis_back_right</rightRearJoint>
-      <wheelSeparation>${base_width}</wheelSeparation>
-      <wheelDiameter>${2*wheel_radius}</wheelDiameter>
-      <robotBaseFrame>base_link</robotBaseFrame>
-      <torque>20</torque>
-      <topicName>cmd_vel</topicName>
-      <broadcastTF>true</broadcastTF>
+    <plugin name="gazebo_ros2_control" filename="libgazebo_ros2_control.so">
+      <parameters>$(find shelfbot)/config/four_wheel_drive_controller.yaml</parameters>
     </plugin>
   </gazebo>

File: urdf/shelfbot.urdf.xacro (robot description, xacro)
@@ -7,5 +7,4 @@
   <xacro:include filename="$(find shelfbot)/urdf/camera.xacro"/>
   <xacro:include filename="$(find shelfbot)/urdf/base_axis.xacro"/>
-  <!-- Fix: Include the Gazebo-specific properties -->
   <xacro:include filename="$(find shelfbot)/urdf/gazebo.urdf.xacro"/>
   <!-- Base Footprint Link -->
@@ -77,4 +76,5 @@
     <origin xyz="0 0 0" rpy="0 0 0"/>
     <axis xyz="0 0 1"/>
+    <limit effort="10" velocity="10"/>
   </joint>
   <joint name="joint_base_axis_front_right" type="continuous">
@@ -83,4 +83,5 @@
     <origin xyz="0 0 0" rpy="0 0 0"/>
     <axis xyz="0 0 1"/>
+    <limit effort="10" velocity="10"/>
   </joint>
   <joint name="joint_base_axis_back_left" type="continuous">
@@ -89,4 +90,5 @@
     <origin xyz="0 0 0" rpy="0 0 0"/>
     <axis xyz="0 0 1"/>
+    <limit effort="10" velocity="10"/>
   </joint>
   <joint name="joint_base_axis_back_right" type="continuous">
@@ -95,4 +97,5 @@
     <origin xyz="0 0 0" rpy="0 0 0"/>
     <axis xyz="0 0 1"/>
+    <limit effort="10" velocity="10"/>
   </joint>
   <!-- Wheels Joints -->
@@ -125,3 +128,29 @@
     <origin xyz="0 0 ${base_height}" rpy="0 0 0"/>
   </joint>
+  <!-- ros2_control -->
+  <ros2_control name="FourWheelDriveSystem" type="system">
+    <hardware>
+      <plugin>shelfbot/FourWheelDriveController</plugin>
+    </hardware>
+    <joint name="joint_base_axis_front_left">
+      <command_interface name="velocity"/>
+      <state_interface name="position"/>
+      <state_interface name="velocity"/>
+    </joint>
+    <joint name="joint_base_axis_front_right">
+      <command_interface name="velocity"/>
+      <state_interface name="position"/>
+      <state_interface name="velocity"/>
+    </joint>
+    <joint name="joint_base_axis_back_left">
+      <command_interface name="velocity"/>
+      <state_interface name="position"/>
+      <state_interface name="velocity"/>
+    </joint>
+    <joint name="joint_base_axis_back_right">
+      <command_interface name="velocity"/>
+      <state_interface name="position"/>
+      <state_interface name="velocity"/>
+    </joint>
+  </ros2_control>
 </robot>

Commit message: Removing transmission elements for now.

File: urdf/gazebo.urdf.xacro (robot description, xacro)
@@ -95,16 +95,4 @@
   <xacro:base_axis_joint_gazebo name="joint_base_axis_back_left"/>
   <xacro:base_axis_joint_gazebo name="joint_base_axis_back_right"/>
-  <xacro:macro name="wheel_transmission" params="name">
-    <transmission name="${name}_transmission">
-      <type>transmission_interface/SimpleTransmission</type>
-      <joint name="${name}">
-        <hardwareInterface>hardware_interface/PositionJointInterface</hardwareInterface>
-      </joint>
-      <actuator name="${name}_motor">
-        <hardwareInterface>hardware_interface/PositionJointInterface</hardwareInterface>
-        <mechanicalReduction>1</mechanicalReduction>
-      </actuator>
-    </transmission>
-  </xacro:macro>
   <gazebo>
     <plugin name="gazebo_ros2_control" filename="libgazebo_ros2_control.so">

Commit message: feat(gazebo): Complete Gazebo simulation setup

File: urdf/gazebo.urdf.xacro (robot description, xacro)
@@ -1,115 +1,48 @@
 <?xml version="1.0"?>
 <robot xmlns:xacro="http://www.ros.org/wiki/xacro">
-  <gazebo reference="base_link">
-    <material>Gazebo/Gold</material>
-  </gazebo>
-  <gazebo reference="indicator_box">
-    <material>Gazebo/Red</material>
-  </gazebo>
-  <xacro:macro name="wheel_gazebo" params="name">
-    <gazebo reference="${name}">
-      <material>Gazebo/Black</material>
-      <mu1>1.8</mu1>
-      <mu2>1.8</mu2>
-      <kp>1000000.0</kp>
-      <kd>100.0</kd>
-      <minDepth>0.001</minDepth>
-      <maxVel>1000.0</maxVel>
-      <fdir1>1 0 0</fdir1>
-      <surface>
-        <friction>
-          <ode>
-            <mu>1.8</mu>
-            <mu2>1.8</mu2>
-            <fdir1>1 0 0</fdir1>
-          </ode>
-        </friction>
-        <contact>
-          <ode>
-            <kp>1e6</kp>
-            <kd>100.0</kd>
-            <max_vel>100.0</max_vel>
-            <min_depth>0.001</min_depth>
-          </ode>
-        </contact>
-      </surface>
+  <xacro:macro name="shelfbot_gazebo">
+    <xacro:arg name="controller_config_file" default=""/>
+    <ros2_control name="GazeboSystem" type="system">
+      <hardware>
+        <plugin>gazebo_ros2_control/GazeboSystem</plugin>
+      </hardware>
+      <joint name="joint_base_axis_front_left">
+        <command_interface name="velocity">
+          <param name="min">-10</param>
+          <param name="max">10</param>
+        </command_interface>
+        <state_interface name="position"/>
+        <state_interface name="velocity"/>
+      </joint>
+      <joint name="joint_base_axis_back_left">
+        <command_interface name="velocity">
+          <param name="min">-10</param>
+          <param name="max">10</param>
+        </command_interface>
+        <state_interface name="position"/>
+        <state_interface name="velocity"/>
+      </joint>
+      <joint name="joint_base_axis_back_right">
+        <command_interface name="velocity">
+          <param name="min">-10</param>
+          <param name="max">10</param>
+        </command_interface>
+        <state_interface name="position"/>
+        <state_interface name="velocity"/>
+      </joint>
+      <joint name="joint_base_axis_front_right">
+        <command_interface name="velocity">
+          <param name="min">-10</param>
+          <param name="max">10</param>
+        </command_interface>
+        <state_interface name="position"/>
+        <state_interface name="velocity"/>
+      </joint>
+    </ros2_control>
+    <gazebo>
+      <plugin name="gazebo_ros2_control" filename="libgazebo_ros2_control.so">
+        <parameters>$(arg controller_config_file)</parameters>
+      </plugin>
     </gazebo>
   </xacro:macro>
-  <xacro:wheel_gazebo name="wheel_front_left"/>
-  <xacro:wheel_gazebo name="wheel_front_right"/>
-  <xacro:wheel_gazebo name="wheel_back_left"/>
-  <xacro:wheel_gazebo name="wheel_back_right"/>
-  <xacro:macro name="base_axis_gazebo" params="name">
-    <gazebo reference="${name}">
-      <material>Gazebo/Red</material>
-    </gazebo>
-  </xacro:macro>
-  <xacro:base_axis_gazebo name="base_axis_front_left"/>
-  <xacro:base_axis_gazebo name="base_axis_front_right"/>
-  <xacro:base_axis_gazebo name="base_axis_back_left"/>
-  <xacro:base_axis_gazebo name="base_axis_back_right"/>
-  <xacro:macro name="motor_gazebo" params="name">
-    <gazebo reference="${name}">
-      <material>Gazebo/Grey</material>
-    </gazebo>
-  </xacro:macro>
-  <xacro:motor_gazebo name="motor_front_left"/>
-  <xacro:motor_gazebo name="motor_front_right"/>
-  <xacro:motor_gazebo name="motor_back_left"/>
-  <xacro:motor_gazebo name="motor_back_right"/>
-  <gazebo reference="camera">
-    <material>Gazebo/Blue</material>
-    <sensor type="camera" name="camera">
-      <update_rate>30.0</update_rate>
-      <camera name="head">
-        <horizontal_fov>1.3962634</horizontal_fov>
-        <image>
-          <width>800</width>
-          <height>600</height>
-          <format>R8G8B8</format>
-        </image>
-        <clip>
-          <near>0.02</near>
-          <far>300</far>
-        </clip>
-        <pose>0 0 0 0 ${pi/2} 0</pose>
-      </camera>
-      <plugin name="camera_controller" filename="libgazebo_ros_camera.so">
-        <alwaysOn>true</alwaysOn>
-        <updateRate>0.0</updateRate>
-        <cameraName>shelfbot/camera</cameraName>
-        <imageTopicName>image_raw</imageTopicName>
-        <cameraInfoTopicName>camera_info</cameraInfoTopicName>
-        <frameName>camera</frameName>
-      </plugin>
-    </sensor>
-  </gazebo>
-  <xacro:macro name="base_axis_joint_gazebo" params="name">
-    <gazebo reference="${name}">
-      <provideFeedback>true</provideFeedback>
-      <implicitSpringDamper>true</implicitSpringDamper>
-    </gazebo>
-  </xacro:macro>
-  <xacro:base_axis_joint_gazebo name="joint_base_axis_front_left"/>
-  <xacro:base_axis_joint_gazebo name="joint_base_axis_front_right"/>
-  <xacro:base_axis_joint_gazebo name="joint_base_axis_back_left"/>
-  <xacro:base_axis_joint_gazebo name="joint_base_axis_back_right"/>
-  <xacro:macro name="wheel_transmission" params="name">
-    <transmission name="${name}_transmission">
-      <type>transmission_interface/SimpleTransmission</type>
-      <joint name="${name}">
-        <hardwareInterface>hardware_interface/PositionJointInterface</hardwareInterface>
-      </joint>
-      <actuator name="${name}_motor">
-        <hardwareInterface>hardware_interface/PositionJointInterface</hardwareInterface>
-        <mechanicalReduction>1</mechanicalReduction>
-      </actuator>
-    </transmission>
-  </xacro:macro>
-  <gazebo>
-    <plugin name="gazebo_ros2_control" filename="libgazebo_ros2_control.so">
-      <robotNamespace>/</robotNamespace>
-      <parameters>$(find shelfbot)/config/four_wheel_drive_controller.yaml</parameters>
-    </plugin>
-  </gazebo>
 </robot>

File: urdf/shelfbot.urdf.xacro (robot description, xacro)
@@ -16,4 +16,5 @@
   <xacro:if value="${'$(arg sim_mode)' == 'gazebo'}">
     <xacro:include filename="$(find shelfbot)/urdf/gazebo.urdf.xacro"/>
+    <xacro:shelfbot_gazebo/>
   </xacro:if>
   <xacro:if value="${'$(arg sim_mode)' == 'isaac'}">
