Commit message: initial implementation using microROS agent path.

File: urdf/real.robot.urdf.xacro (robot description, xacro)
@@ -1,8 +1,31 @@
 <?xml version="1.0"?>
 <robot xmlns:xacro="http://www.ros.org/wiki/xacro">
-<hardware>
-  <plugin>shelfbot/FourWheelDriveHardwareInterface</plugin>
-  <param name="communication_type">rest</param>
-  <param name="base_url">http://shelfbot.local/</param>
-</hardware>
+  <!-- Declare arguments that this file expects to receive -->
+  <xacro:arg name="communication_type" default="rest"/>
+  <xacro:arg name="base_url" default="http://shelfbot.local/"/>
+  <!-- Define the ros2_control system for the real robot -->
+  <ros2_control name="FourWheelDriveSystem" type="system">
+    <hardware>
+      <plugin>shelfbot/FourWheelDriveHardwareInterface</plugin>
+      <!-- Use the passed-in arguments to set the parameters -->
+      <param name="communication_type">$(arg communication_type)</param>
+      <param name="base_url">$(arg base_url)</param>
+    </hardware>
+    <joint name="joint_base_axis_front_left">
+      <command_interface name="position"/>
+      <state_interface name="position"/>
+    </joint>
+    <joint name="joint_base_axis_front_right">
+      <command_interface name="position"/>
+      <state_interface name="position"/>
+    </joint>
+    <joint name="joint_base_axis_back_left">
+      <command_interface name="position"/>
+      <state_interface name="position"/>
+    </joint>
+    <joint name="joint_base_axis_back_right">
+      <command_interface name="position"/>
+      <state_interface name="position"/>
+    </joint>
+  </ros2_control>
 </robot>

File: urdf/shelfbot.urdf.xacro (robot description, xacro)
@@ -1,4 +1,5 @@
 <?xml version="1.0"?>
 <robot xmlns:xacro="http://www.ros.org/wiki/xacro" name="shelfbot">
+  <!-- Include all the component parts of the robot -->
   <xacro:include filename="$(find shelfbot)/urdf/common_properties.xacro"/>
   <xacro:include filename="$(find shelfbot)/urdf/motor.xacro"/>
@@ -7,5 +8,9 @@
   <xacro:include filename="$(find shelfbot)/urdf/base_axis.xacro"/>
   <xacro:include filename="$(find shelfbot)/urdf/box.xacro"/>
+  <!-- Declare the arguments that will be passed in from the launch file -->
   <xacro:arg name="sim_mode" default="gazebo"/>
+  <xacro:arg name="communication_type" default="rest"/>
+  <xacro:arg name="base_url" default="http://shelfbot.local/"/>
+  <!-- Include the correct hardware interface based on sim_mode -->
   <xacro:if value="${'$(arg sim_mode)' == 'gazebo'}">
     <xacro:include filename="$(find shelfbot)/urdf/gazebo.urdf.xacro"/>
@@ -14,7 +19,12 @@
     <xacro:include filename="$(find shelfbot)/urdf/isaac.sim.urdf.xacro"/>
   </xacro:if>
+  <!-- When using the real robot, include the real.robot.urdf.xacro and pass the communication arguments down to it -->
   <xacro:if value="${'$(arg sim_mode)' == 'real'}">
-    <xacro:include filename="$(find shelfbot)/urdf/real.robot.urdf.xacro"/>
+    <xacro:include filename="$(find shelfbot)/urdf/real.robot.urdf.xacro">
+      <xacro:arg name="communication_type" value="$(arg communication_type)"/>
+      <xacro:arg name="base_url" value="$(arg base_url)"/>
+    </xacro:include>
   </xacro:if>
+  <!-- Robot Physical Structure -->
   <link name="base_footprint"/>
   <link name="base_link">
@@ -127,39 +137,3 @@
     <origin xyz="0 0 ${base_height}" rpy="${-pi/2} 0 0"/>
   </joint>
-<ros2_control name="FourWheelDriveSystem" type="system">
-    <xacro:if value="${'$(arg sim_mode)' == 'gazebo'}">
-        <hardware>
-            <plugin>gazebo_ros2_control/GazeboSystem</plugin>
-        </hardware>
-    </xacro:if>
-    <xacro:if value="${'$(arg sim_mode)' == 'isaac'}">
-        <hardware>
-            <plugin>shelfbot/FourWheelDriveHardwareInterface</plugin>
-            <param name="communication_type">mock</param>
-        </hardware>
-    </xacro:if>
-    <xacro:if value="${'$(arg sim_mode)' == 'real'}">
-        <hardware>
-            <plugin>shelfbot/FourWheelDriveHardwareInterface</plugin>
-            <param name="communication_type">rest</param>
-            <param name="base_url">http://shelfbot.local/</param>
-        </hardware>
-    </xacro:if>
-    <joint name="joint_base_axis_front_left">
-        <command_interface name="position"/>
-        <state_interface name="position"/>
-    </joint>
-    <joint name="joint_base_axis_front_right">
-        <command_interface name="position"/>
-        <state_interface name="position"/>
-    </joint>
-    <joint name="joint_base_axis_back_left">
-        <command_interface name="position"/>
-        <state_interface name="position"/>
-    </joint>
-    <joint name="joint_base_axis_back_right">
-        <command_interface name="position"/>
-        <state_interface name="position"/>
-    </joint>
-</ros2_control>
 </robot>

Commit message: Refactor: Remove simulation and simplify communication layers
Removes Gazebo simulation and communication libraries (REST, serial, mock) to focus on the real robot with micro-ROS. Updates all configurations, launch files, and documentation accordingly.

File: urdf/real.robot.urdf.xacro (robot description, xacro)
@@ -2,5 +2,5 @@
 <robot xmlns:xacro="http://www.ros.org/wiki/xacro">
   <!-- Declare arguments with default values -->
-  <xacro:arg name="communication_type" default="rest"/>
+  <xacro:arg name="communication_type" default="microros"/>
   <xacro:arg name="base_url" default="http://shelfbot.local/"/>
   <ros2_control name="FourWheelDriveSystem" type="system">

File: urdf/shelfbot.urdf.xacro (robot description, xacro)
@@ -10,22 +10,10 @@
   <xacro:include filename="$(find shelfbot)/urdf/ultrasonic_sensor.xacro"/>
   <!-- Declare the arguments that will be passed in from the launch file -->
-  <xacro:arg name="sim_mode" default="gazebo"/>
-  <xacro:arg name="communication_type" default="rest"/>
   <xacro:arg name="base_url" default="http://shelfbot.local/"/>
-  <!-- Include the correct hardware interface based on sim_mode -->
-  <xacro:if value="${'$(arg sim_mode)' == 'gazebo'}">
-    <xacro:include filename="$(find shelfbot)/urdf/gazebo.urdf.xacro"/>
-    <xacro:shelfbot_gazebo/>
-  </xacro:if>
-  <xacro:if value="${'$(arg sim_mode)' == 'isaac'}">
-    <xacro:include filename="$(find shelfbot)/urdf/isaac.sim.urdf.xacro"/>
-  </xacro:if>
-  <!-- When using the real robot, include the real.robot.urdf.xacro and pass the communication arguments down to it -->
-  <xacro:if value="${'$(arg sim_mode)' == 'real'}">
-    <xacro:include filename="$(find shelfbot)/urdf/real.robot.urdf.xacro">
-      <xacro:arg name="communication_type" value="$(arg communication_type)"/>
-      <xacro:arg name="base_url" value="$(arg base_url)"/>
-    </xacro:include>
-  </xacro:if>
+  <!-- Set properties that will be used by the included real.robot.urdf.xacro -->
+  <xacro:property name="communication_type" value="microros"/>
+  <xacro:property name="base_url" value="$(arg base_url)"/>
+  <!-- When using the real robot, include the real.robot.urdf.xacro -->
+  <xacro:include filename="$(find shelfbot)/urdf/real.robot.urdf.xacro"/>
   <!-- Robot Physical Structure -->
   <link name="base_footprint"/>
