Commit message: adjusting motor positions and kinematics to match the sketch.

File: urdf/camera.xacro (robot description, xacro)
@@ -1,14 +1,34 @@
 <?xml version="1.0"?>
 <robot xmlns:xacro="http://www.ros.org/wiki/xacro">
-  <xacro:macro name="camera" params="name width length height radius">
+  <!--
+    Camera body + optical frame.
+    params:
+      name   - link name (also used as prefix for child links/joints)
+      width  - x dimension of camera box
+      length - y dimension of camera box
+      height - z dimension of camera box  (lens face is at +Z of this link)
+    Coordinate convention after joint_camera (rpy="-pi/2 0 0") is applied:
+      camera_link +Z = base_link +Y (forward, optical axis)
+      camera_link +X = base_link +X (right)
+      camera_link +Y = base_link -Z (down)
+    camera_link is therefore already in ROS optical convention.
+    The _optical_frame child adds the standard rpy="-pi/2 0 -pi/2" transform
+    so that image_pipeline, rtabmap and other tools that look for an optical
+    frame find one with the expected parent→child relationship.
+    The frame_id in camera_info messages must be "${name}_optical_frame".
+    Update the camera_publisher frame_id parameter accordingly.
+  -->
+  <xacro:macro name="camera" params="name width length height">
+    <!-- Camera body -->
     <link name="${name}">
       <visual>
-        <origin xyz="0 0 ${height/2}"/>
+        <origin xyz="0 0 ${height/2}" rpy="0 0 0"/>
         <geometry>
           <box size="${width} ${length} ${height}"/>
         </geometry>
+        <material name="metallic_dark_lead"/>
       </visual>
       <collision>
-        <origin xyz="0 0 ${height/2}"/>
+        <origin xyz="0 0 ${height/2}" rpy="0 0 0"/>
         <geometry>
           <box size="${width} ${length} ${height}"/>
@@ -21,4 +41,19 @@
       </inertial>
     </link>
+    <!--
+      Optical frame.
+      Positioned at the lens face (z = height of the camera body).
+      rpy="-pi/2 0 -pi/2" is the standard ROS transform from a camera body
+      link to its optical frame: converts from body convention (X fwd, Y left,
+      Z up) to optical convention (Z fwd, X right, Y down).
+      All camera_info and image messages should use "${name}_optical_frame"
+      as their frame_id.
+    -->
+    <link name="${name}_optical_frame"/>
+    <joint name="joint_${name}_optical" type="fixed">
+      <parent link="${name}"/>
+      <child link="${name}_optical_frame"/>
+      <origin xyz="0 0 ${height}" rpy="-1.5708 0 -1.5708"/>
+    </joint>
   </xacro:macro>
 </robot>

File: urdf/shelfbot.urdf.xacro (robot description, xacro)
@@ -1,92 +1,32 @@
 <?xml version="1.0"?>
 <robot xmlns:xacro="http://www.ros.org/wiki/xacro" name="shelfbot">
-  <!-- Load all properties from the YAML file -->
-  <xacro:property name="config_file" value="$(find shelfbot)/config/four_wheel_drive_controller.yaml" />
-  <xacro:property name="config" value="${xacro.load_yaml(config_file)}" />
-  <!-- Define materials -->
-  <material name="golden_brown">
-    <color rgba="0.87 0.72 0.53 1.0"/>
-  </material>
-  <material name="metallic_dark_lead">
-    <color rgba="0.33 0.33 0.33 1.0"/>
-  </material>
-  <material name="dark_red">
-    <color rgba="0.55 0.0 0.0 1.0"/>
-  </material>
-  <material name="metallic_gray">
-    <color rgba="0.66 0.66 0.66 1.0"/>
-  </material>
-  <material name="red">
-    <color rgba="1.0 0.0 0.0 1.0"/>
-  </material>
-  <material name="blue">
-    <color rgba="0.0 0.0 1.0 1.0"/>
-  </material>
-  <material name="light_grey">
-    <color rgba="0.8 0.8 0.8 1.0"/>
-  </material>
-  <!-- Define properties from the loaded YAML -->
-  <xacro:property name="base_width" value="${config['four_wheel_drive_controller']['ros__parameters']['base_width']}"/>
-  <xacro:property name="base_length" value="${config['four_wheel_drive_controller']['ros__parameters']['base_length']}"/>
-  <xacro:property name="base_height" value="${config['four_wheel_drive_controller']['ros__parameters']['base_height']}"/>
-  <xacro:property name="base_mass" value="${config['four_wheel_drive_controller']['ros__parameters']['base_mass']}"/>
-  <xacro:property name="motor_radius" value="${config['four_wheel_drive_controller']['ros__parameters']['motor_radius']}"/>
-  <xacro:property name="motor_length" value="${config['four_wheel_drive_controller']['ros__parameters']['motor_length']}"/>
-  <xacro:property name="motor_mass" value="${config['four_wheel_drive_controller']['ros__parameters']['motor_mass']}"/>
-  <xacro:property name="wheel_radius" value="${config['four_wheel_drive_controller']['ros__parameters']['wheel_radius']}"/>
-  <xacro:property name="wheel_width" value="${config['four_wheel_drive_controller']['ros__parameters']['wheel_width']}"/>
-  <xacro:property name="wheel_mass" value="${config['four_wheel_drive_controller']['ros__parameters']['wheel_mass']}"/>
-  <xacro:property name="camera_width" value="${config['four_wheel_drive_controller']['ros__parameters']['camera_width']}"/>
-  <xacro:property name="camera_length" value="${config['four_wheel_drive_controller']['ros__parameters']['camera_length']}"/>
-  <xacro:property name="camera_height" value="${config['four_wheel_drive_controller']['ros__parameters']['camera_height']}"/>
-  <xacro:property name="camera_lens_radius" value="${config['four_wheel_drive_controller']['ros__parameters']['camera_lens_radius']}"/>
-  <xacro:property name="camera_mount_height" value="${config['four_wheel_drive_controller']['ros__parameters']['camera_mount_height']}"/>
-  <xacro:property name="camera_mass" value="${config['four_wheel_drive_controller']['ros__parameters']['camera_mass']}"/>
-  <xacro:property name="base_axis_radius" value="${config['four_wheel_drive_controller']['ros__parameters']['base_axis_radius']}"/>
-  <xacro:property name="base_axis_length" value="${config['four_wheel_drive_controller']['ros__parameters']['base_axis_length']}"/>
-  <xacro:property name="base_axis_mass" value="${config['four_wheel_drive_controller']['ros__parameters']['base_axis_mass']}"/>
-  <xacro:property name="gear_ratio" value="${config['four_wheel_drive_controller']['ros__parameters']['gear_ratio']}"/>
-  <xacro:property name="box_x_size" value="${config['four_wheel_drive_controller']['ros__parameters']['box_x_size']}"/>
-  <xacro:property name="box_y_size" value="${config['four_wheel_drive_controller']['ros__parameters']['box_y_size']}"/>
-  <xacro:property name="box_z_size" value="${config['four_wheel_drive_controller']['ros__parameters']['box_z_size']}"/>
-  <xacro:property name="box_mass" value="${config['four_wheel_drive_controller']['ros__parameters']['box_mass']}"/>
-  <xacro:property name="box_inertia" value="${config['four_wheel_drive_controller']['ros__parameters']['box_inertia']}"/>
-  <xacro:property name="ultrasonic_pcb_x_size" value="${config['four_wheel_drive_controller']['ros__parameters']['ultrasonic_pcb_x_size']}"/>
-  <xacro:property name="ultrasonic_pcb_y_size" value="${config['four_wheel_drive_controller']['ros__parameters']['ultrasonic_pcb_y_size']}"/>
-  <xacro:property name="ultrasonic_pcb_z_size" value="${config['four_wheel_drive_controller']['ros__parameters']['ultrasonic_pcb_z_size']}"/>
-  <xacro:property name="ultrasonic_collision_z_size" value="${config['four_wheel_drive_controller']['ros__parameters']['ultrasonic_collision_z_size']}"/>
-  <xacro:property name="ultrasonic_mass" value="${config['four_wheel_drive_controller']['ros__parameters']['ultrasonic_mass']}"/>
-  <xacro:property name="ultrasonic_transducer_radius" value="${config['four_wheel_drive_controller']['ros__parameters']['ultrasonic_transducer_radius']}"/>
-  <xacro:property name="ultrasonic_transducer_length" value="${config['four_wheel_drive_controller']['ros__parameters']['ultrasonic_transducer_length']}"/>
-  <xacro:property name="ultrasonic_transducer_x_offset" value="${config['four_wheel_drive_controller']['ros__parameters']['ultrasonic_transducer_x_offset']}"/>
-  <xacro:property name="ultrasonic_z_offset" value="${config['four_wheel_drive_controller']['ros__parameters']['ultrasonic_z_offset']}"/>
-  <xacro:property name="joint_damping" value="${config['four_wheel_drive_controller']['ros__parameters']['joint_damping']}"/>
-  <xacro:property name="joint_friction" value="${config['four_wheel_drive_controller']['ros__parameters']['joint_friction']}"/>
-  <!-- Define inertia macros -->
-  <xacro:macro name="cylinder_inertia" params="m r h">
-    <inertia ixx="${m*(3*r*r+h*h)/12}" ixy="0" ixz="0"
-             iyy="${m*(3*r*r+h*h)/12}" iyz="0"
-             izz="${m*r*r/2}"/>
-  </xacro:macro>
-  <xacro:macro name="box_inertia" params="m x y z">
-    <inertia ixx="${m*(y*y+z*z)/12}" ixy="0" ixz="0"
-             iyy="${m*(x*x+z*z)/12}" iyz="0"
-             izz="${m*(x*x+y*y)/12}"/>
-  </xacro:macro>
-  <!-- Include the component parts of the robot -->
+  <!-- ═══════════════════════════════════════════════════════════════════
+       Single source of truth: all materials, properties and inertia
+       macros live in common_properties.xacro.  Nothing is duplicated here.
+       ═══════════════════════════════════════════════════════════════════ -->
+  <xacro:include filename="$(find shelfbot)/urdf/common_properties.xacro"/>
+  <!-- ═══════════════════════════════════════════════════════════════════
+       Component macros
+       ═══════════════════════════════════════════════════════════════════ -->
   <xacro:include filename="$(find shelfbot)/urdf/motor.xacro"/>
   <xacro:include filename="$(find shelfbot)/urdf/wheel.xacro"/>
   <xacro:include filename="$(find shelfbot)/urdf/camera.xacro"/>
   <xacro:include filename="$(find shelfbot)/urdf/base_axis.xacro"/>
-  <xacro:include filename="$(find shelfbot)/urdf/box.xacro"/>
   <xacro:include filename="$(find shelfbot)/urdf/ultrasonic_sensor.xacro"/>
-  <!-- Declare the arguments that will be passed in from the launch file -->
-  <xacro:arg name="base_url" default="http://shelfbot.local/"/>
-  <xacro:arg name="communication_type" default="${str(config['controller_manager']['ros__parameters']['hardware_interface']['communication_type'])}"/>
-  <xacro:arg name="wheel_separation" default="${str(config['four_wheel_drive_controller']['ros__parameters']['wheel_separation'])}"/>
-  <xacro:arg name="wheel_radius" default="${str(config['four_wheel_drive_controller']['ros__parameters']['wheel_radius'])}"/>
-  <!-- When using the real robot, include the real.robot.urdf.xacro -->
+  <!-- ═══════════════════════════════════════════════════════════════════
+       Launch-file arguments (config is already loaded by common_properties)
+       ═══════════════════════════════════════════════════════════════════ -->
+  <xacro:arg name="base_url"            default="http://shelfbot.local/"/>
+  <xacro:arg name="communication_type"  default="${str(config['controller_manager']['ros__parameters']['hardware_interface']['communication_type'])}"/>
+  <xacro:arg name="wheel_separation"    default="${str(config['four_wheel_drive_controller']['ros__parameters']['wheel_separation'])}"/>
+  <xacro:arg name="wheel_radius"        default="${str(config['four_wheel_drive_controller']['ros__parameters']['wheel_radius'])}"/>
+  <!-- ═══════════════════════════════════════════════════════════════════
+       ros2_control hardware interface (real robot)
+       ═══════════════════════════════════════════════════════════════════ -->
   <xacro:include filename="$(find shelfbot)/urdf/real.robot.urdf.xacro"/>
-  <!-- Robot Physical Structure -->
+  <!-- ═══════════════════════════════════════════════════════════════════
+       Robot physical structure
+       ═══════════════════════════════════════════════════════════════════ -->
+  <!-- Root link — no inertial, no visual: required by REP 120 -->
   <link name="base_footprint"/>
   <link name="base_link">
@@ -108,41 +48,48 @@
     </inertial>
   </link>
+  <!-- base_footprint sits on the ground; base_link centre is raised by
+       half its height plus one wheel radius -->
   <joint name="joint_base_footprint" type="fixed">
     <parent link="base_footprint"/>
     <child link="base_link"/>
-    <origin xyz="0 0 ${base_height / 2 + wheel_radius}" rpy="0 0 0"/>
-  </joint>
-  <xacro:motor name="motor_front_left" length="${motor_length}" radius="${motor_radius}"/>
+    <origin xyz="0 0 ${base_height/2 + wheel_radius}" rpy="0 0 0"/>
+  </joint>
+  <!-- ── Motors (fixed to base_link) ───────────────────────────────── -->
+  <xacro:motor name="motor_front_left"  length="${motor_length}" radius="${motor_radius}"/>
   <xacro:motor name="motor_front_right" length="${motor_length}" radius="${motor_radius}"/>
-  <xacro:motor name="motor_back_left" length="${motor_length}" radius="${motor_radius}"/>
-  <xacro:motor name="motor_back_right" length="${motor_length}" radius="${motor_radius}"/>
-  <xacro:base_axis name="base_axis_front_left" length="${base_axis_length}" radius="${base_axis_radius}"/>
+  <xacro:motor name="motor_back_left"   length="${motor_length}" radius="${motor_radius}"/>
+  <xacro:motor name="motor_back_right"  length="${motor_length}" radius="${motor_radius}"/>
+  <!-- Left motors: rpy="pi/2 0 pi"   → shaft exits toward -Y (left side)
+       Right motors: rpy="-pi/2 0 0"  → shaft exits toward +Y (right side) -->
+  <joint name="joint_motor_front_left" type="fixed">
+    <parent link="base_link"/>
+    <child link="motor_front_left"/>
+    <origin xyz="${-base_width/2 + motor_length} ${base_length/2 - 0.075} 0"
+            rpy="${pi/2} 0 ${pi}"/>
+  </joint>
+  <joint name="joint_motor_front_right" type="fixed">
+    <parent link="base_link"/>
+    <child link="motor_front_right"/>
+    <origin xyz="${base_width/2 - motor_length} ${base_length/2 - 0.075} 0"
+            rpy="${-pi/2} 0 0"/>
+  </joint>
+  <joint name="joint_motor_back_left" type="fixed">
+    <parent link="base_link"/>
+    <child link="motor_back_left"/>
+    <origin xyz="${-base_width/2 + motor_length} ${-base_length/2 + 0.075} 0"
+            rpy="${pi/2} 0 ${pi}"/>
+  </joint>
+  <joint name="joint_motor_back_right" type="fixed">
+    <parent link="base_link"/>
+    <child link="motor_back_right"/>
+    <origin xyz="${base_width/2 - motor_length} ${-base_length/2 + 0.075} 0"
+            rpy="${-pi/2} 0 0"/>
+  </joint>
+  <!-- ── Drive axles (continuous, controlled by ros2_control) ──────── -->
+  <xacro:base_axis name="base_axis_front_left"  length="${base_axis_length}" radius="${base_axis_radius}"/>
   <xacro:base_axis name="base_axis_front_right" length="${base_axis_length}" radius="${base_axis_radius}"/>
-  <xacro:base_axis name="base_axis_back_left" length="${base_axis_length}" radius="${base_axis_radius}"/>
-  <xacro:base_axis name="base_axis_back_right" length="${base_axis_length}" radius="${base_axis_radius}"/>
-  <xacro:wheel name="wheel_front_left" radius="${wheel_radius}" width="${wheel_width}"/>
-  <xacro:wheel name="wheel_front_right" radius="${wheel_radius}" width="${wheel_width}"/>
-  <xacro:wheel name="wheel_back_left" radius="${wheel_radius}" width="${wheel_width}"/>
-  <xacro:wheel name="wheel_back_right" radius="${wheel_radius}" width="${wheel_width}"/>
-  <joint name="joint_motor_front_left" type="fixed">
-    <parent link="base_link"/>
-    <child link="motor_front_left"/>
-    <origin xyz="${-base_width / 2 + motor_length} ${base_length / 2 - 0.075} 0" rpy="${pi/2} 0 ${pi}"/>
-  </joint>
-  <joint name="joint_motor_front_right" type="fixed">
-    <parent link="base_link"/>
-    <child link="motor_front_right"/>
-    <origin xyz="${base_width / 2 - motor_length} ${base_length / 2 - 0.075} 0" rpy="${-pi/2} 0 0"/>
-  </joint>
-  <joint name="joint_motor_back_left" type="fixed">
-    <parent link="base_link"/>
-    <child link="motor_back_left"/>
-    <origin xyz="${-base_width / 2 + motor_length} ${-base_length / 2 + 0.075} 0" rpy="${pi/2} 0 ${pi}"/>
-  </joint>
-  <joint name="joint_motor_back_right" type="fixed">
-    <parent link="base_link"/>
-    <child link="motor_back_right"/>
-    <origin xyz="${base_width / 2 - motor_length} ${-base_length / 2 + 0.075} 0" rpy="${-pi/2} 0 0"/>
-  </joint>
+  <xacro:base_axis name="base_axis_back_left"   length="${base_axis_length}" radius="${base_axis_radius}"/>
+  <xacro:base_axis name="base_axis_back_right"  length="${base_axis_length}" radius="${base_axis_radius}"/>
+  <!-- Left axles rotate around local +X, offset by -pi/2 from motor frame -->
   <joint name="joint_base_axis_front_left" type="continuous">
     <parent link="motor_front_left"/>
@@ -173,31 +120,54 @@
     <dynamics damping="${joint_damping}" friction="${joint_friction}"/>
   </joint>
+  <!-- ── Wheels (fixed to axles) ───────────────────────────────────── -->
+  <xacro:wheel name="wheel_front_left"  radius="${wheel_radius}" width="${wheel_width}"/>
+  <xacro:wheel name="wheel_front_right" radius="${wheel_radius}" width="${wheel_width}"/>
+  <xacro:wheel name="wheel_back_left"   radius="${wheel_radius}" width="${wheel_width}"/>
+  <xacro:wheel name="wheel_back_right"  radius="${wheel_radius}" width="${wheel_width}"/>
+  <!-- Wheel inner face aligns with axle tip:
+       offset = base_width/2 - motor_length (must equal base_axis_length) -->
   <joint name="joint_wheel_front_left" type="fixed">
     <parent link="base_axis_front_left"/>
     <child link="wheel_front_left"/>
-    <origin xyz="${base_width / 2 - motor_length} 0 0" rpy="0 0 0"/>
+    <origin xyz="${base_width/2 - motor_length} 0 0" rpy="0 0 0"/>
   </joint>
   <joint name="joint_wheel_front_right" type="fixed">
     <parent link="base_axis_front_right"/>
     <child link="wheel_front_right"/>
-    <origin xyz="${base_width / 2 - motor_length} 0 0" rpy="0 0 0"/>
+    <origin xyz="${base_width/2 - motor_length} 0 0" rpy="0 0 0"/>
   </joint>
   <joint name="joint_wheel_back_left" type="fixed">
     <parent link="base_axis_back_left"/>
     <child link="wheel_back_left"/>
-    <origin xyz="${base_width / 2 - motor_length} 0 0" rpy="0 0 0"/>
+    <origin xyz="${base_width/2 - motor_length} 0 0" rpy="0 0 0"/>
   </joint>
   <joint name="joint_wheel_back_right" type="fixed">
     <parent link="base_axis_back_right"/>
     <child link="wheel_back_right"/>
-    <origin xyz="${base_width / 2 - motor_length} 0 0" rpy="0 0 0"/>
-  </joint>
-  <xacro:camera name="camera_link" width="${camera_width}" length="${camera_length}" height="${camera_height}" radius="${camera_lens_radius}"/>
+    <origin xyz="${base_width/2 - motor_length} 0 0" rpy="0 0 0"/>
+  </joint>
+  <!-- ── Camera ────────────────────────────────────────────────────── -->
+  <!--
+    camera.xacro creates two links: camera_link and camera_link_optical_frame.
+    After joint_camera (rpy="-pi/2 0 0") camera_link axes in base_link space:
+      +Z = base_link +Y (forward / optical axis)
+      +X = base_link +X (right)
+      +Y = base_link -Z (down)
+    camera_link is therefore already in ROS optical convention.
+    camera_link_optical_frame adds the standard rpy="-pi/2 0 -pi/2" child for
+    image_pipeline / rtabmap compatibility.
+    The camera_publisher frame_id parameter must be "camera_link_optical_frame".
+  -->
+  <xacro:camera name="camera_link"
+                width="${camera_width}"
+                length="${camera_length}"
+                height="${camera_height}"/>
   <joint name="joint_camera" type="fixed">
     <parent link="base_link"/>
     <child link="camera_link"/>
+    <!-- Centred on top face of base_link, facing forward (+Y) -->
     <origin xyz="0 0 ${base_height}" rpy="${-pi/2} 0 0"/>
   </joint>
-  <!-- Ultrasonic Sensors (3-Front, 3-Back Configuration) -->
+  <!-- ── Ultrasonic sensors (3 front, 3 back) ──────────────────────── -->
   <xacro:ultrasonic_sensor name="us_front_center"/>
   <xacro:ultrasonic_sensor name="us_front_left_corner"/>
@@ -206,33 +176,41 @@
   <xacro:ultrasonic_sensor name="us_back_left_corner"/>
   <xacro:ultrasonic_sensor name="us_back_right_corner"/>
+  <!-- Front sensors: rpy="0 pi/2 angle" orients PCB face outward -->
   <joint name="joint_us_front_center" type="fixed">
     <parent link="base_link"/>
     <child link="us_front_center"/>
-    <origin xyz="0 ${base_length / 2} ${ultrasonic_z_offset}" rpy="0 ${pi/2} ${pi/2}"/>
+    <origin xyz="0 ${base_length/2} ${ultrasonic_z_offset}"
+            rpy="0 ${pi/2} ${pi/2}"/>
   </joint>
   <joint name="joint_us_front_left_corner" type="fixed">
     <parent link="base_link"/>
     <child link="us_front_left_corner"/>
-    <origin xyz="${base_width / 4} ${base_length / 2} ${ultrasonic_z_offset}" rpy="0 ${pi/2} ${pi/4}"/>
+    <origin xyz="${base_width/4} ${base_length/2} ${ultrasonic_z_offset}"
+            rpy="0 ${pi/2} ${pi/4}"/>
   </joint>
   <joint name="joint_us_front_right_corner" type="fixed">
     <parent link="base_link"/>
     <child link="us_front_right_corner"/>
-    <origin xyz="${-base_width / 4} ${base_length / 2} ${ultrasonic_z_offset}" rpy="0 ${pi/2} ${3*pi/4}"/>
-  </joint>
+    <origin xyz="${-base_width/4} ${base_length/2} ${ultrasonic_z_offset}"
+            rpy="0 ${pi/2} ${3*pi/4}"/>
+  </joint>
+  <!-- Back sensors -->
   <joint name="joint_us_back_center" type="fixed">
     <parent link="base_link"/>
     <child link="us_back_center"/>
-    <origin xyz="0 ${-base_length / 2} ${ultrasonic_z_offset}" rpy="0 ${pi/2} ${-pi/2}"/>
+    <origin xyz="0 ${-base_length/2} ${ultrasonic_z_offset}"
+            rpy="0 ${pi/2} ${-pi/2}"/>
   </joint>
   <joint name="joint_us_back_left_corner" type="fixed">
     <parent link="base_link"/>
     <child link="us_back_left_corner"/>
-    <origin xyz="${base_width / 4} ${-base_length / 2} ${ultrasonic_z_offset}" rpy="0 ${pi/2} ${-pi/4}"/>
+    <origin xyz="${base_width/4} ${-base_length/2} ${ultrasonic_z_offset}"
+            rpy="0 ${pi/2} ${-pi/4}"/>
   </joint>
   <joint name="joint_us_back_right_corner" type="fixed">
     <parent link="base_link"/>
     <child link="us_back_right_corner"/>
-    <origin xyz="${-base_width / 4} ${-base_length / 2} ${ultrasonic_z_offset}" rpy="0 ${pi/2} ${-3*pi/4}"/>
+    <origin xyz="${-base_width/4} ${-base_length/2} ${ultrasonic_z_offset}"
+            rpy="0 ${pi/2} ${-3*pi/4}"/>
   </joint>
 </robot>
