Commit message: Troubleshooting the continuous type of joint.

File: urdf/shelfbot.urdf.xacro (robot description, xacro)
@@ -6,6 +6,4 @@
   <xacro:include filename="$(find shelfbot)/urdf/wheel.xacro"/>
   <xacro:include filename="$(find shelfbot)/urdf/camera.xacro"/>
-  <xacro:include filename="$(find shelfbot)/urdf/fixed_joint.xacro"/>
-  <xacro:include filename="$(find shelfbot)/urdf/revolute_joint.xacro"/>
   <xacro:include filename="$(find shelfbot)/urdf/base_axis.xacro"/>
   <!-- Base Footprint Link -->
@@ -20,6 +18,10 @@
     </visual>
   </link>
-  <!-- Modified joint to raise base_link -->
-  <xacro:fixed_joint name="joint_base_footprint" parent="base_footprint" child="base_link" origin_xyz="0 0 ${base_height / 2 + wheel_radius}" origin_rpy="0 0 0"/>
+  <!-- Joint to raise base_link -->
+  <joint name="joint_base_footprint" type="fixed">
+    <parent link="base_footprint"/>
+    <child link="base_link"/>
+    <origin xyz="0 0 ${base_height / 2 + wheel_radius}" rpy="0 0 0"/>
+  </joint>
   <!-- Base Axes -->
   <xacro:base_axis name="base_axis_front_left" length="${base_axis_length}" radius="${base_axis_radius}"/>
@@ -28,8 +30,24 @@
   <xacro:base_axis name="base_axis_back_right" length="${base_axis_length}" radius="${base_axis_radius}"/>
   <!-- Base Axes Joints -->
-  <xacro:fixed_joint name="joint_base_axis_front_left" parent="base_link" child="base_axis_front_left" origin_xyz="${-base_width / 2} ${base_length / 2} 0" origin_rpy="0 ${pi/2} 0"/>
-  <xacro:fixed_joint name="joint_base_axis_front_right" parent="base_link" child="base_axis_front_right" origin_xyz="${base_width / 2} ${base_length / 2} 0" origin_rpy="0 ${pi/2} 0"/>
-  <xacro:fixed_joint name="joint_base_axis_back_left" parent="base_link" child="base_axis_back_left" origin_xyz="${-base_width / 2} ${-base_length / 2} 0" origin_rpy="0 ${pi/2} 0"/>
-  <xacro:fixed_joint name="joint_base_axis_back_right" parent="base_link" child="base_axis_back_right" origin_xyz="${base_width / 2} ${-base_length / 2} 0" origin_rpy="0 ${pi/2} 0"/>
+  <joint name="joint_base_axis_front_left" type="fixed">
+    <parent link="base_link"/>
+    <child link="base_axis_front_left"/>
+    <origin xyz="${-base_width / 2} ${base_length / 2} 0" rpy="0 ${pi/2} 0"/>
+  </joint>
+  <joint name="joint_base_axis_front_right" type="fixed">
+    <parent link="base_link"/>
+    <child link="base_axis_front_right"/>
+    <origin xyz="${base_width / 2} ${base_length / 2} 0" rpy="0 ${pi/2} 0"/>
+  </joint>
+  <joint name="joint_base_axis_back_left" type="fixed">
+    <parent link="base_link"/>
+    <child link="base_axis_back_left"/>
+    <origin xyz="${-base_width / 2} ${-base_length / 2} 0" rpy="0 ${pi/2} 0"/>
+  </joint>
+  <joint name="joint_base_axis_back_right" type="fixed">
+    <parent link="base_link"/>
+    <child link="base_axis_back_right"/>
+    <origin xyz="${base_width / 2} ${-base_length / 2} 0" rpy="0 ${pi/2} 0"/>
+  </joint>
   <!-- Motors -->
   <xacro:motor name="motor_front_left" length="${motor_length}" radius="${motor_radius}" mass="1.0" ixx="0.01" ixy="0.0" ixz="0.0" iyy="0.01" iyz="0.0" izz="0.01"/>
@@ -38,8 +56,24 @@
   <xacro:motor name="motor_back_right" length="${motor_length}" radius="${motor_radius}" mass="1.0" ixx="0.01" ixy="0.0" ixz="0.0" iyy="0.01" iyz="0.0" izz="0.01"/>
   <!-- Motor Joints -->
-  <xacro:fixed_joint name="joint_motor_front_left" parent="base_axis_front_left" child="motor_front_left" origin_xyz="0 0 0" origin_rpy="0 0 0"/>
-  <xacro:fixed_joint name="joint_motor_front_right" parent="base_axis_front_right" child="motor_front_right" origin_xyz="0 0 0" origin_rpy="0 0 0"/>
-  <xacro:fixed_joint name="joint_motor_back_left" parent="base_axis_back_left" child="motor_back_left" origin_xyz="0 0 0" origin_rpy="0 0 0"/>
-  <xacro:fixed_joint name="joint_motor_back_right" parent="base_axis_back_right" child="motor_back_right" origin_xyz="0 0 0" origin_rpy="0 0 0"/>
+  <joint name="joint_motor_front_left" type="fixed">
+    <parent link="base_axis_front_left"/>
+    <child link="motor_front_left"/>
+    <origin xyz="0 0 0" rpy="0 0 0"/>
+  </joint>
+  <joint name="joint_motor_front_right" type="fixed">
+    <parent link="base_axis_front_right"/>
+    <child link="motor_front_right"/>
+    <origin xyz="0 0 0" rpy="0 0 0"/>
+  </joint>
+  <joint name="joint_motor_back_left" type="fixed">
+    <parent link="base_axis_back_left"/>
+    <child link="motor_back_left"/>
+    <origin xyz="0 0 0" rpy="0 0 0"/>
+  </joint>
+  <joint name="joint_motor_back_right" type="fixed">
+    <parent link="base_axis_back_right"/>
+    <child link="motor_back_right"/>
+    <origin xyz="0 0 0" rpy="0 0 0"/>
+  </joint>
   <!-- Wheels -->
   <xacro:wheel name="wheel_front_left" radius="${wheel_radius}" width="${wheel_width}"/>
@@ -48,11 +82,31 @@
   <xacro:wheel name="wheel_back_right" radius="${wheel_radius}" width="${wheel_width}"/>
   <!-- Wheels Joints -->
-  <xacro:fixed_joint name="joint_wheel_front_left" parent="base_axis_front_left" child="wheel_front_left" origin_xyz="0 0 -${motor_length/2}" origin_rpy="0 0 0"/>
-  <xacro:fixed_joint name="joint_wheel_front_right" parent="base_axis_front_right" child="wheel_front_right" origin_xyz="0 0 ${motor_length/2}" origin_rpy="0 0 0"/>
-  <xacro:fixed_joint name="joint_wheel_back_left" parent="base_axis_back_left" child="wheel_back_left" origin_xyz="0 0 -${motor_length/2}" origin_rpy="0 0 0"/>
-  <xacro:fixed_joint name="joint_wheel_back_right" parent="base_axis_back_right" child="wheel_back_right" origin_xyz="0 0 ${motor_length/2}" origin_rpy="0 0 0"/>
+  <joint name="joint_wheel_front_left" type="fixed">
+    <parent link="base_axis_front_left"/>
+    <child link="wheel_front_left"/>
+    <origin xyz="0 0 -${motor_length/2}" rpy="0 0 0"/>
+  </joint>
+  <joint name="joint_wheel_front_right" type="fixed">
+    <parent link="base_axis_front_right"/>
+    <child link="wheel_front_right"/>
+    <origin xyz="0 0 ${motor_length/2}" rpy="0 0 0"/>
+  </joint>
+  <joint name="joint_wheel_back_left" type="fixed">
+    <parent link="base_axis_back_left"/>
+    <child link="wheel_back_left"/>
+    <origin xyz="0 0 -${motor_length/2}" rpy="0 0 0"/>
+  </joint>
+  <joint name="joint_wheel_back_right" type="fixed">
+    <parent link="base_axis_back_right"/>
+    <child link="wheel_back_right"/>
+    <origin xyz="0 0 ${motor_length/2}" rpy="0 0 0"/>
+  </joint>
   <!-- Camera -->
   <xacro:camera name="camera" width="${camera_width}" length="${camera_length}" height="${camera_height}" radius="${camera_lens_radius}"/>
   <!-- Camera Joint -->
-  <xacro:fixed_joint name="joint_camera" parent="base_link" child="camera" origin_xyz="0 0 ${base_height}" origin_rpy="0 0 0"/>
+  <joint name="joint_camera" type="fixed">
+    <parent link="base_link"/>
+    <child link="camera"/>
+    <origin xyz="0 0 ${base_height}" rpy="0 0 0"/>
+  </joint>
 </robot>

Commit message: Fixing launchers.

File: urdf/shelfbot.urdf.xacro (robot description, xacro)
@@ -65,5 +65,5 @@
     <child link="base_axis_front_left"/>
     <origin xyz="0 0 0" rpy="0 0 0"/>
-    <axis xyz="0 1 0"/>
+    <axis xyz="0 0 1"/>
     <limit lower="-3.14159" upper="3.14159" effort="100" velocity="1.0"/>
     <dynamics damping="0.1" friction="0.1"/>
@@ -73,5 +73,5 @@
     <child link="base_axis_front_right"/>
     <origin xyz="0 0 0" rpy="0 0 0"/>
-    <axis xyz="0 1 0"/>
+    <axis xyz="0 0 1"/>
     <limit lower="-3.14159" upper="3.14159" effort="100" velocity="1.0"/>
     <dynamics damping="0.1" friction="0.1"/>
@@ -81,5 +81,5 @@
     <child link="base_axis_back_left"/>
     <origin xyz="0 0 0" rpy="0 0 0"/>
-    <axis xyz="0 1 0"/>
+    <axis xyz="0 0 1"/>
     <limit lower="-3.14159" upper="3.14159" effort="100" velocity="1.0"/>
     <dynamics damping="0.1" friction="0.1"/>
@@ -89,5 +89,5 @@
     <child link="base_axis_back_right"/>
     <origin xyz="0 0 0" rpy="0 0 0"/>
-    <axis xyz="0 1 0"/>
+    <axis xyz="0 0 1"/>
     <limit lower="-3.14159" upper="3.14159" effort="100" velocity="1.0"/>
     <dynamics damping="0.1" friction="0.1"/>

Commit message: Adding real robot and isaac sim configuration.

File: urdf/shelfbot.urdf.xacro (robot description, xacro)
@@ -6,6 +6,15 @@
   <xacro:include filename="$(find shelfbot)/urdf/camera.xacro"/>
   <xacro:include filename="$(find shelfbot)/urdf/base_axis.xacro"/>
-  <xacro:include filename="$(find shelfbot)/urdf/gazebo.urdf.xacro"/>
   <xacro:include filename="$(find shelfbot)/urdf/box.xacro"/>
+  <xacro:property name="sim_mode" value="gazebo"/>
+  <xacro:if value="${sim_mode == 'gazebo'}">
+    <xacro:include filename="$(find shelfbot)/urdf/gazebo.urdf.xacro"/>
+  </xacro:if>
+  <xacro:if value="${sim_mode == 'isaac'}">
+    <xacro:include filename="$(find shelfbot)/urdf/isaac.sim.urdf.xacro"/>
+  </xacro:if>
+  <xacro:if value="${sim_mode == 'real'}">
+    <xacro:include filename="$(find shelfbot)/urdf/real.robot.urdf.xacro"/>
+  </xacro:if>
   <link name="base_footprint"/>
   <link name="base_link">

Commit message: Implementing hardware_interface::SystemInterface overrides.

File: urdf/shelfbot.urdf.xacro (robot description, xacro)
@@ -7,14 +7,42 @@
   <xacro:include filename="$(find shelfbot)/urdf/base_axis.xacro"/>
   <xacro:include filename="$(find shelfbot)/urdf/box.xacro"/>
-  <xacro:property name="sim_mode" value="gazebo"/>
-  <xacro:if value="${sim_mode == 'gazebo'}">
+  <xacro:arg name="sim_mode" default="gazebo"/>
+  <xacro:if value="${'$(arg sim_mode)' == 'gazebo'}">
     <xacro:include filename="$(find shelfbot)/urdf/gazebo.urdf.xacro"/>
   </xacro:if>
-  <xacro:if value="${sim_mode == 'isaac'}">
+  <xacro:if value="${'$(arg sim_mode)' == 'isaac'}">
     <xacro:include filename="$(find shelfbot)/urdf/isaac.sim.urdf.xacro"/>
   </xacro:if>
-  <xacro:if value="${sim_mode == 'real'}">
+  <xacro:if value="${'$(arg sim_mode)' == 'real'}">
     <xacro:include filename="$(find shelfbot)/urdf/real.robot.urdf.xacro"/>
   </xacro:if>
+  <ros2_control name="FourWheelDriveSystem" type="system">
+    <xacro:if value="${'$(arg sim_mode)' == 'gazebo'}">
+      <hardware>
+        <plugin>gazebo_ros2_control/GazeboSystem</plugin>
+      </hardware>
+    </xacro:if>
+    <xacro:if value="${'$(arg sim_mode)' != 'gazebo'}">
+      <hardware>
+        <plugin>shelfbot/FourWheelDriveController</plugin>
+      </hardware>
+    </xacro:if>
+    <joint name="joint_base_axis_front_left">
+      <command_interface name="position"/>
+      <state_interface name="position"/>
+    </joint>
+    <joint name="joint_base_axis_front_right">
+      <command_interface name="position"/>
+      <state_interface name="position"/>
+    </joint>
+    <joint name="joint_base_axis_back_left">
+      <command_interface name="position"/>
+      <state_interface name="position"/>
+    </joint>
+    <joint name="joint_base_axis_back_right">
+      <command_interface name="position"/>
+      <state_interface name="position"/>
+    </joint>
+  </ros2_control>
   <link name="base_footprint"/>
   <link name="base_link">
@@ -128,24 +156,3 @@
     <origin xyz="0 0 ${base_height}" rpy="${-pi/2} 0 0"/>
   </joint>
-  <ros2_control name="FourWheelDriveSystem" type="system">
-    <hardware>
-      <plugin>gazebo_ros2_control/GazeboSystem</plugin>
-    </hardware>
-    <joint name="joint_base_axis_front_left">
-      <command_interface name="position"/>
-      <state_interface name="position"/>
-    </joint>
-    <joint name="joint_base_axis_front_right">
-      <command_interface name="position"/>
-      <state_interface name="position"/>
-    </joint>
-    <joint name="joint_base_axis_back_left">
-      <command_interface name="position"/>
-      <state_interface name="position"/>
-    </joint>
-    <joint name="joint_base_axis_back_right">
-      <command_interface name="position"/>
-      <state_interface name="position"/>
-    </joint>
-  </ros2_control>
 </robot>

Commit message: Changing the order for readability.

File: urdf/shelfbot.urdf.xacro (robot description, xacro)
@@ -17,32 +17,4 @@
     <xacro:include filename="$(find shelfbot)/urdf/real.robot.urdf.xacro"/>
   </xacro:if>
-  <ros2_control name="FourWheelDriveSystem" type="system">
-    <xacro:if value="${'$(arg sim_mode)' == 'gazebo'}">
-      <hardware>
-        <plugin>gazebo_ros2_control/GazeboSystem</plugin>
-      </hardware>
-    </xacro:if>
-    <xacro:if value="${'$(arg sim_mode)' != 'gazebo'}">
-      <hardware>
-        <plugin>shelfbot/FourWheelDriveController</plugin>
-      </hardware>
-    </xacro:if>
-    <joint name="joint_base_axis_front_left">
-      <command_interface name="position"/>
-      <state_interface name="position"/>
-    </joint>
-    <joint name="joint_base_axis_front_right">
-      <command_interface name="position"/>
-      <state_interface name="position"/>
-    </joint>
-    <joint name="joint_base_axis_back_left">
-      <command_interface name="position"/>
-      <state_interface name="position"/>
-    </joint>
-    <joint name="joint_base_axis_back_right">
-      <command_interface name="position"/>
-      <state_interface name="position"/>
-    </joint>
-  </ros2_control>
   <link name="base_footprint"/>
   <link name="base_link">
@@ -69,12 +41,12 @@
     <origin xyz="0 0 ${base_height / 2 + wheel_radius}" rpy="0 0 0"/>
   </joint>
+  <xacro:motor name="motor_front_left" length="${motor_length}" radius="${motor_radius}"/>
+  <xacro:motor name="motor_front_right" length="${motor_length}" radius="${motor_radius}"/>
+  <xacro:motor name="motor_back_left" length="${motor_length}" radius="${motor_radius}"/>
+  <xacro:motor name="motor_back_right" length="${motor_length}" radius="${motor_radius}"/>
   <xacro:base_axis name="base_axis_front_left" length="${base_axis_length}" radius="${base_axis_radius}"/>
   <xacro:base_axis name="base_axis_front_right" length="${base_axis_length}" radius="${base_axis_radius}"/>
   <xacro:base_axis name="base_axis_back_left" length="${base_axis_length}" radius="${base_axis_radius}"/>
   <xacro:base_axis name="base_axis_back_right" length="${base_axis_length}" radius="${base_axis_radius}"/>
-  <xacro:motor name="motor_front_left" length="${motor_length}" radius="${motor_radius}"/>
-  <xacro:motor name="motor_front_right" length="${motor_length}" radius="${motor_radius}"/>
-  <xacro:motor name="motor_back_left" length="${motor_length}" radius="${motor_radius}"/>
-  <xacro:motor name="motor_back_right" length="${motor_length}" radius="${motor_radius}"/>
   <xacro:wheel name="wheel_front_left" radius="${wheel_radius}" width="${wheel_width}"/>
   <xacro:wheel name="wheel_front_right" radius="${wheel_radius}" width="${wheel_width}"/>
@@ -156,3 +128,31 @@
     <origin xyz="0 0 ${base_height}" rpy="${-pi/2} 0 0"/>
   </joint>
+  <ros2_control name="FourWheelDriveSystem" type="system">
+    <xacro:if value="${'$(arg sim_mode)' == 'gazebo'}">
+      <hardware>
+        <plugin>gazebo_ros2_control/GazeboSystem</plugin>
+      </hardware>
+    </xacro:if>
+    <xacro:if value="${'$(arg sim_mode)' != 'gazebo'}">
+      <hardware>
+        <plugin>shelfbot/FourWheelDriveController</plugin>
+      </hardware>
+    </xacro:if>
+    <joint name="joint_base_axis_front_left">
+      <command_interface name="position"/>
+      <state_interface name="position"/>
+    </joint>
+    <joint name="joint_base_axis_front_right">
+      <command_interface name="position"/>
+      <state_interface name="position"/>
+    </joint>
+    <joint name="joint_base_axis_back_left">
+      <command_interface name="position"/>
+      <state_interface name="position"/>
+    </joint>
+    <joint name="joint_base_axis_back_right">
+      <command_interface name="position"/>
+      <state_interface name="position"/>
+    </joint>
+  </ros2_control>
 </robot>

Commit message: fix(rviz): Correct odometry calculation and robot model orientation
This commit resolves several issues that caused incorrect visualization of the robot's odometry and model in RViz.

- Corrected the micro-ROS subscriber to listen for /shelfbot_firmware/motor_positions to receive hardware state updates.
- Fixed the odometry calculation in FourWheelDriveOdometry to correctly compute forward distance and rotation from wheel positions.
- Resolved a frame ID mismatch between the /odom topic and the TF broadcast, setting both to use base_footprint.
- Rotated the base_link in the URDF to align the robot's visual "front" with the standard X-axis.
- Added a 180-degree offset to the final odometry orientation to make the RViz arrow point backward as requested for this project's specific visualization needs.
- Updated the launch file to use a specific RViz configuration and reduce log spam from the state publisher and control nodes.

File: urdf/shelfbot.urdf.xacro (robot description, xacro)
@@ -49,5 +49,5 @@
     <parent link="base_footprint"/>
     <child link="base_link"/>
-    <origin xyz="0 0 ${base_height / 2 + wheel_radius}" rpy="0 0 0"/>
+    <origin xyz="0 0 ${base_height / 2 + wheel_radius}" rpy="0 0 -1.57079632679"/>
   </joint>
   <xacro:motor name="motor_front_left" length="${motor_length}" radius="${motor_radius}"/>

Commit message: feat(robot): Overhaul launch system and RTAB-Map.

File: urdf/shelfbot.urdf.xacro (robot description, xacro)
@@ -133,8 +133,8 @@
     <origin xyz="${base_axis_length/2} 0 0" rpy="0 0 0"/>
   </joint>
-  <xacro:camera name="camera" width="${camera_width}" length="${camera_length}" height="${camera_height}" radius="${camera_lens_radius}"/>
+  <xacro:camera name="camera_link" width="${camera_width}" length="${camera_length}" height="${camera_height}" radius="${camera_lens_radius}"/>
   <joint name="joint_camera" type="fixed">
     <parent link="base_link"/>
-    <child link="camera"/>
+    <child link="camera_link"/>
     <origin xyz="0 0 ${base_height}" rpy="${-pi/2} 0 0"/>
   </joint>

Commit message: fix(odom): Correct odometry orientation and remove interfering nodes
- Restores the -90 degree rotation to the `joint_base_footprint` in the
  URDF. This is necessary to align the "sideways" `base_link` model
  with the ROS standard "X-forward" `base_footprint`.
- Removes hardcoded static transform publishers from the Nav2 launch
  file that were conflicting with the `robot_state_publisher`.
- Removes an erroneous +180 degree rotation from the odometry C++
  code that was causing an incorrect static offset.

File: urdf/shelfbot.urdf.xacro (robot description, xacro)
@@ -111,5 +111,5 @@
     <parent link="base_footprint"/>
     <child link="base_link"/>
-    <origin xyz="0 0 ${base_height / 2 + wheel_radius}" rpy="0 0 -1.57079632679"/>
+    <origin xyz="0 0 ${base_height / 2 + wheel_radius}" rpy="0 0 0"/>
   </joint>
   <xacro:motor name="motor_front_left" length="${motor_length}" radius="${motor_radius}"/>

Commit message: creating launcher and node for lidar scan.

File: urdf/shelfbot.urdf.xacro (robot description, xacro)
@@ -13,4 +13,5 @@
   <xacro:include filename="$(find shelfbot)/urdf/camera.xacro"/>
   <xacro:include filename="$(find shelfbot)/urdf/base_axis.xacro"/>
+  <xacro:include filename="$(find shelfbot)/urdf/lidar_sensor.xacro"/>
   <xacro:include filename="$(find shelfbot)/urdf/ultrasonic_sensor.xacro"/>
   <!-- ═══════════════════════════════════════════════════════════════════
@@ -169,4 +170,11 @@
     <origin xyz="0 0 ${base_height}" rpy="${-pi/2} 0 0"/>
   </joint>
+  <xacro:lidar_sensor name="laser_link"/>
+  <joint name="joint_laser" type="fixed">
+    <parent link="base_link"/>
+    <child link="laser_link"/>
+    <!-- Centred on top face; adjust z if the lidar sits above/below the camera -->
+    <origin xyz="0 0 ${base_height}" rpy="0 0 0"/>
+  </joint>
   <!-- ── Ultrasonic sensors (3 front, 3 back) ──────────────────────── -->
   <xacro:ultrasonic_sensor name="us_front_center"/>

Commit message: eks initial configuration and adding to filtered /odom.

File: urdf/shelfbot.urdf.xacro (robot description, xacro)
@@ -49,10 +49,8 @@
     </inertial>
   </link>
-  <!-- base_footprint sits on the ground; base_link centre is raised by
-       half its height plus one wheel radius -->
   <joint name="joint_base_footprint" type="fixed">
     <parent link="base_footprint"/>
     <child link="base_link"/>
-    <origin xyz="0 0 ${base_height/2 + wheel_radius}" rpy="0 0 0"/>
+    <origin xyz="0 0 ${base_height/2 + wheel_radius}" rpy="0 0 ${-pi/2}"/>
   </joint>
   <!-- ── Motors (fixed to base_link) ───────────────────────────────── -->
