Commit message: Align lidar frame with robot front

File: urdf/lidar_sensor.xacro (robot description, xacro)
@@ -3,6 +3,8 @@
   <!--
     Minimal laser_link for the LYDSTO LDS02RR lidar.
-    Mounted flat on top of base_link, centred, facing up.
-    Adjust xyz/rpy to match physical placement.
+    Mounted flat with the scan plane parallel to the floor.  Per REP 103,
+    LaserScan angle 0 is along laser_link +X and positive angles rotate toward
+    +Y.  The mounting joint in shelfbot.urdf.xacro is responsible for placing
+    +X along the robot's physical forward direction.
   -->
   <xacro:macro name="lidar_sensor" params="name">

File: urdf/shelfbot.urdf.xacro (robot description, xacro)
@@ -160,8 +160,12 @@
   </joint>
   <xacro:lidar_sensor name="laser_link"/>
+  <!-- The physical robot front is base_link +Y (mapped to base_footprint +X by
+       joint_base_footprint's -pi/2 yaw).  LaserScan angle 0 is laser_link +X,
+       so yaw laser_link +90 deg relative to base_link and place it at the
+       front tip of the chassis. -->
   <joint name="joint_laser" type="fixed">
     <parent link="base_link"/>
     <child link="laser_link"/>
-    <origin xyz="0 0 ${base_height}" rpy="0 0 0"/>
+    <origin xyz="0 ${base_length/2} ${base_height}" rpy="0 0 ${pi/2}"/>
   </joint>
   <!-- ── Ultrasonic sensors (3 front, 3 back) ──────────────────────── -->

Commit message: Flip lidar yaw correction

File: urdf/lidar_sensor.xacro (robot description, xacro)
@@ -3,6 +3,8 @@
   <!--
     Minimal laser_link for the LYDSTO LDS02RR lidar.
-    Mounted flat on top of base_link, centred, facing up.
-    Adjust xyz/rpy to match physical placement.
+    Mounted flat with the scan plane parallel to the floor.  Per REP 103,
+    LaserScan angle 0 is along laser_link +X and positive angles rotate toward
+    +Y.  The mounting joint in shelfbot.urdf.xacro is responsible for applying
+    the measured yaw correction needed by the real scanner.
   -->
   <xacro:macro name="lidar_sensor" params="name">

File: urdf/shelfbot.urdf.xacro (robot description, xacro)
@@ -160,8 +160,12 @@
   </joint>
   <xacro:lidar_sensor name="laser_link"/>
+  <!-- The physical robot front is base_link +Y (mapped to base_footprint +X by
+       joint_base_footprint's -pi/2 yaw).  The real lidar scan ordering is
+       inverted relative to the previous +pi/2 model, so yaw laser_link -90 deg
+       relative to base_link and keep it at the front tip of the chassis. -->
   <joint name="joint_laser" type="fixed">
     <parent link="base_link"/>
     <child link="laser_link"/>
-    <origin xyz="0 0 ${base_height}" rpy="0 0 0"/>
+    <origin xyz="0 ${base_length/2} ${base_height}" rpy="0 0 ${-pi/2}"/>
   </joint>
   <!-- ── Ultrasonic sensors (3 front, 3 back) ──────────────────────── -->

Commit message: Flip lidar yaw correction (#23)

File: urdf/lidar_sensor.xacro (robot description, xacro)
@@ -5,6 +5,6 @@
     Mounted flat with the scan plane parallel to the floor.  Per REP 103,
     LaserScan angle 0 is along laser_link +X and positive angles rotate toward
-    +Y.  The mounting joint in shelfbot.urdf.xacro is responsible for placing
-    +X along the robot's physical forward direction.
+    +Y.  The mounting joint in shelfbot.urdf.xacro is responsible for applying
+    the measured yaw correction needed by the real scanner.
   -->
   <xacro:macro name="lidar_sensor" params="name">

File: urdf/shelfbot.urdf.xacro (robot description, xacro)
@@ -161,11 +161,11 @@
   <xacro:lidar_sensor name="laser_link"/>
   <!-- The physical robot front is base_link +Y (mapped to base_footprint +X by
-       joint_base_footprint's -pi/2 yaw).  LaserScan angle 0 is laser_link +X,
-       so yaw laser_link +90 deg relative to base_link and place it at the
-       front tip of the chassis. -->
+       joint_base_footprint's -pi/2 yaw).  The real lidar scan ordering is
+       inverted relative to the previous +pi/2 model, so yaw laser_link -90 deg
+       relative to base_link and keep it at the front tip of the chassis. -->
   <joint name="joint_laser" type="fixed">
     <parent link="base_link"/>
     <child link="laser_link"/>
-    <origin xyz="0 ${base_length/2} ${base_height}" rpy="0 0 ${pi/2}"/>
+    <origin xyz="0 ${base_length/2} ${base_height}" rpy="0 0 ${-pi/2}"/>
   </joint>
   <!-- ── Ultrasonic sensors (3 front, 3 back) ──────────────────────── -->
